Commit message: 初始化项目

File: aubo_ros2_ws/src/aubo_ros2_driver/aubo_description/urdf/xacro/inc/aubo_ros2.xacro (robot description, xacro)
@@ -504,4 +504,5 @@
   </joint>
   <!-- /////////////////////////////////   e5 pedestal_Link   ////////////////////////////////////// -->
+  <!-- 修改：将 base_link 作为根链接，pedestal_Link 作为 base_link 的子链接 -->
   <link name="pedestal_Link">
     <visual>
@@ -511,10 +512,14 @@
     </visual>
   </link>
+  <!-- 修改：反转关节关系，使 base_link 成为父链接，pedestal_Link 成为子链接 -->
+  <!-- 注意：偏移量需要反转（从 base_link 到 pedestal_Link 是向下 0.503m） -->
   <joint name="pedestal_joint" type="fixed">
-    <parent link="pedestal_Link"/>
-    <child link="base_link"/>
-    <origin xyz="0.0 0.0 0.503" rpy="0.0 0.0 0.0" />
-  </joint>
- <!-- /////////////////////////////////   world   ////////////////////////////////////// -->
+    <parent link="base_link"/>
+    <child link="pedestal_Link"/>
+    <origin xyz="0.0 0.0 -0.503" rpy="0.0 0.0 0.0" />
+  </joint>
+  <!-- 注释掉 world 链接和 world_joint，使 base_link 成为根链接 -->
+  <!-- 如果需要 world 坐标系，可以通过 TF 静态变换发布 -->
+  <!--
   <link name="world" />
   <joint name="world_joint" type="fixed">
@@ -523,4 +528,5 @@
     <origin xyz="0.0 0.0 0.0" rpy="0.0 0.0 0.0" />
   </joint>
+  -->
   <!-- /////////////////////////////////   gazebo color   ////////////////////////////////////// -->
   <gazebo reference="pedestal_Link">

Commit message: 自动手眼标定数据计算误差计算5mm验证完成

File: aubo_ros2_ws/src/aubo_ros2_driver/aubo_description/urdf/xacro/inc/aubo_ros2.xacro (robot description, xacro)
@@ -503,4 +503,29 @@
     <origin xyz="0.0 0.0 0.0" rpy="0.0 0.0 0.0" />
   </joint>
+  <!-- /////////////////////////////////   Tool Center Point (TCP) with Camera   ////////////////////////////////////// -->
+  <!-- 添加 TCP 偏移以匹配手眼标定的位姿 -->
+  <!-- Z 轴偏移 0.024m (24mm) 用于补偿相机或工具的偏移 -->
+  <link name="tool_center_point">
+    <inertial>
+      <origin xyz="0 0 0" rpy="0 0 0" />
+      <mass value="0.001" />
+      <inertia ixx="0.000001" ixy="0" ixz="0" iyy="0.000001" iyz="0" izz="0.000001" />
+    </inertial>
+    <visual>
+      <origin xyz="0 0 0" rpy="0 0 0"/>
+      <geometry>
+        <sphere radius="0.005"/>
+      </geometry>
+      <material name="">
+        <color rgba="1 0 0 1" />  <!-- 红色标记 TCP -->
+      </material>
+    </visual>
+  </link>
+  <joint name="ee_to_tcp_joint" type="fixed">
+    <parent link="ee_link" />
+    <child link="tool_center_point" />
+    <!-- TCP with no offset - Accurate MoveIt2 TF tree for hand-eye calibration -->
+    <origin xyz="0.0 0.0 0.0" rpy="0.0 0.0 0.0" />
+  </joint>
   <!-- /////////////////////////////////   e5 pedestal_Link   ////////////////////////////////////// -->
   <!-- 修改：将 base_link 作为根链接，pedestal_Link 作为 base_link 的子链接 -->

Commit message: 深度阈值模板匹配抓取完成

File: aubo_ros2_ws/src/aubo_ros2_driver/aubo_description/urdf/xacro/inc/aubo_ros2.xacro (robot description, xacro)
@@ -1,515 +1,15 @@
 <?xml version="1.0"?>
-<robot name="aubo_e5" xmlns:xacro="http://ros.org/wiki/xacro">
- <!-- Defining the colors used in this robot -->
-    <material name="Black">
-        <color rgba="0 0 0 1"/>
-    </material>
-    <material name="White">
-        <color rgba="1 1 1 1"/>
-    </material>
-    <material name="Blue">
-        <color rgba="0 0 1 1"/>
-    </material>
-    <material name="Red">
-        <color rgba="1 0 0 1"/>
-    </material>
-    <material name="Grey">
-        <color rgba="0.96 0.96 0.96 1"/>
-    </material>
-    <!-- Constants -->
-    <xacro:property name="M_PI" value="3.14159"/>
-    <!--/////////////////// DYNAMICS PARAM //////////////////////-->
-    <xacro:macro name="I5_Shoulder_Inertia">
-        <origin xyz="0.0 0.006 -0.002"
-                rpy="0 0 0" />
-        <mass value="5.05" />
-        <inertia ixx="0.0148"
-                 ixy="0"
-                 ixz="0"
-                 iyy="0.0143"
-                 iyz="-0.0"
-                 izz="0.0095" />
-    </xacro:macro>
-    <xacro:macro name="I5_UpperArm_Inertia">
-        <origin xyz="0.304 0.0 -0.03"
-                rpy="0 0 0" />
-        <mass value="11.90" />
-        <inertia ixx="0.0305"
-                 ixy="0"
-                 ixz="0"
-                 iyy="0.4505"
-                 iyz="0"
-                 izz="0.0095" />
-    </xacro:macro>
-    <xacro:macro name="I5_ForeArm_Inertia">
-        <origin xyz="0.415 0.0 0.0992"
-                rpy="0 0 0" />
-        <mass  value="3.3" />
-        <inertia ixx="0.0033"
-                 ixy="0"
-                 ixz="0.0009"
-                 iyy="0.0575"
-                 iyz="0"
-                 izz="0.0565" />
-    </xacro:macro>
-    <xacro:macro name="I5_Wrist1_Inertia">
-        <origin xyz="0.0 0.0028 -0.003"
-                rpy="0 0 0" />
-        <mass value="1.62" />
-        <inertia ixx="0.0023"
-                 ixy="0"
-                 ixz="0"
-                 iyy="0.0013"
-                 iyz="0.0"
-                 izz="0.0022" />
-    </xacro:macro>
-    <xacro:macro name="I5_Wrist2_Inertia">
-        <origin xyz="0.0 -0.0028 -0.003"
-                rpy="0 0 0" />
-        <mass value="1.62" />
-        <inertia ixx="0.0023"
-                 ixy="0"
-                 ixz="0"
-                 iyy="0.0013"
-                 iyz="0.0"
-                 izz="0.0022" />
-    </xacro:macro>
-    <xacro:macro name="I5_Wrist3_Inertia">
-        <origin xyz="0.0 0.0 -0.0071"
-                rpy="0 0 0" />
-        <mass value="0.40" />
-        <inertia ixx="0.013939"
-                 ixy="0"
-                 ixz="0"
-                 iyy="0.013988"
-                 iyz="0.0"
-                 izz="0.0224092" />
-    </xacro:macro>
-    <!--/////////////////////////////// BASE_LINK ////////////////////////////////////-->
-   <link
-    name="base_link">
-    <inertial>
-      <origin
-        xyz="4.2454E-05 -1.2043E-08 0.020702"
-        rpy="0 0 0" />
-      <mass
-        value="0.80619" />
-      <inertia
-        ixx="0.0013215"
-        ixy="2.5362E-09"
-        ixz="-1.4252E-05"
-        iyy="0.0013301"
-        iyz="-1.0084E-10"
-        izz="0.0023301" />
-    </inertial>
-    <visual>
-      <origin
-        xyz="0 0 0"
-        rpy="0 0 0" />
-      <geometry>
-        <mesh
-          filename="package://aubo_description/meshes/aubo_e5/visual/base_link.DAE" />
-      </geometry>
-      <material
-        name="">
-        <color
-          rgba="1 1 1 1" />
-      </material>
-    </visual>
-    <collision>
-      <origin
-        xyz="0 0 0"
-        rpy="0 0 0" />
-      <geometry>
-        <mesh
-          filename="package://aubo_description/meshes/aubo_e5/collision/base_link.STL" />
-      </geometry>
-    </collision>
-  </link>
-  <link
-    name="shoulder_Link">
-    <inertial>
-      <origin
-        xyz="-2.1059E-08 0.0083051 0.065103"
-        rpy="0 0 0" />
-      <mass
-        value="1.5715" />
-      <inertia
-        ixx="0.0030796"
-        ixy="6.3642E-08"
-        ixz="1.9408E-08"
-        iyy="0.0028016"
-        iyz="-0.00021308"
-        izz="0.0031979" />
-    </inertial>
-    <visual>
-      <origin
-        xyz="0 0 0"
-        rpy="0 0 0" />
-      <geometry>
-        <mesh
-          filename="package://aubo_description/meshes/aubo_e5/visual/shoulder_Link.DAE" />
-      </geometry>
-      <material
-        name="">
-        <color
-          rgba="1 1 1 1" />
-      </material>
-    </visual>
-    <collision>
-      <origin
-        xyz="0 0 0"
-        rpy="0 0 0" />
-      <geometry>
-        <mesh
-          filename="package://aubo_description/meshes/aubo_e5/collision/shoulder_Link.STL" />
-      </geometry>
-    </collision>
-  </link>
-  <joint
-    name="shoulder_joint"
-    type="revolute">
-    <origin
-      xyz="0 0 0.0495"
-      rpy="0 0 -3.1234" />
-    <parent
-      link="base_link" />
-    <child
-      link="shoulder_Link" />
-    <axis
-      xyz="0 0 1" />
-    <limit
-      lower="-3.05"
-      upper="3.05"
-      effort="0"
-      velocity="0" />
-  </joint>
-  <link
-    name="upperArm_Link">
-    <inertial>
-      <origin
-        xyz="0.204 -0.00063844 0.057604"
-        rpy="0 0 0" />
-      <mass
-        value="4.9786" />
-      <inertia
-        ixx="0.0075025"
-        ixy="3.8877E-05"
-        ixz="-1.4653E-08"
-        iyy="0.019967"
-        iyz="-4.6361E-06"
-        izz="0.020135" />
-    </inertial>
-    <visual>
-      <origin
-        xyz="0 0 0"
-        rpy="0 0 0" />
-      <geometry>
-        <mesh
-          filename="package://aubo_description/meshes/aubo_e5/visual/upperArm_Link.DAE" />
-      </geometry>
-      <material
-        name="">
-        <color
-          rgba="1 1 1 1" />
-      </material>
-    </visual>
-    <collision>
-      <origin
-        xyz="0 0 0"
-        rpy="0 0 0" />
-      <geometry>
-        <mesh
-          filename="package://aubo_description/meshes/aubo_e5/collision/upperArm_Link.STL" />
-      </geometry>
-    </collision>
-  </link>
-  <joint
-    name="upperArm_joint"
-    type="revolute">
-    <origin
-      xyz="0 0.0786 0.0708"
-      rpy="-1.5708 -1.5708 0" />
-    <parent
-      link="shoulder_Link" />
-    <child
-      link="upperArm_Link" />
-    <axis
-      xyz="0 0 1" />
-    <limit
-      lower="-3.05"
-      upper="3.05"
-      effort="0"
-      velocity="0" />
-  </joint>
-  <link
-    name="foreArm_Link">
-    <inertial>
-      <origin
-        xyz="0.18368 0.00064681 0.055339"
-        rpy="0 0 0" />
-      <mass
-        value="2.2775" />
-      <inertia
-        ixx="0.00182"
-        ixy="-2.5051E-05"
-        ixz="-8.9044E-05"
-        iyy="0.0088861"
-        iyz="-1.3488E-06"
-        izz="0.0089876" />
-    </inertial>
-    <visual>
-      <origin
-        xyz="0 0 0"
-        rpy="0 0 0" />
-      <geometry>
-        <mesh
-          filename="package://aubo_description/meshes/aubo_e5/visual/foreArm_Link.DAE" />
-      </geometry>
-      <material
-        name="">
-        <color
-          rgba="1 1 1 1" />
-      </material>
-    </visual>
-    <collision>
-      <origin
-        xyz="0 0 0"
-        rpy="0 0 0" />
-      <geometry>
-        <mesh
-          filename="package://aubo_description/meshes/aubo_e5/collision/foreArm_Link.STL" />
-      </geometry>
-    </collision>
-  </link>
-  <joint
-    name="foreArm_joint"
-    type="revolute">
-    <origin
-      xyz="0.408 -0.0012767 0.0002"
-      rpy="3.1416 0 0" />
-    <parent
-      link="upperArm_Link" />
-    <child
-      link="foreArm_Link" />
-    <axis
-      xyz="0 0 1" />
-    <limit
-      lower="-3.05"
-      upper="3.05"
-      effort="0"
-      velocity="0" />
-  </joint>
-  <link
-    name="wrist1_Link">
-    <inertial>
-      <origin
-        xyz="-5.5568E-06 0.006024 0.051377"
-        rpy="0 0 0" />
-      <mass
-        value="0.47808" />
-      <inertia
-        ixx="0.00043634"
-        ixy="-6.0507E-11"
-        ixz="3.0917E-08"
-        iyy="0.00042786"
-        iyz="-3.1316E-05"
-        izz="0.00038517" />
-    </inertial>
-    <visual>
-      <origin
-        xyz="0 0 0"
-        rpy="0 0 0" />
-      <geometry>
-        <mesh
-          filename="package://aubo_description/meshes/aubo_e5/visual/wrist1_Link.DAE" />
-      </geometry>
-      <material
-        name="">
-        <color
-          rgba="1 1 1 1" />
-      </material>
-    </visual>
-    <collision>
-      <origin
-        xyz="0 0 0"
-        rpy="0 0 0" />
-      <geometry>
-        <mesh
-          filename="package://aubo_description/meshes/aubo_e5/collision/wrist1_Link.STL" />
-      </geometry>
-    </collision>
-  </link>
-  <joint
-    name="wrist1_joint"
-    type="revolute">
-    <origin
-      xyz="0.3736 -8.9586E-05 0.015624"
-      rpy="3.1415 0.03325 1.5708" />
-    <parent
-      link="foreArm_Link" />
-    <child
-      link="wrist1_Link" />
-    <axis
-      xyz="0 0 1" />
-    <limit
-      lower="-3.05"
-      upper="3.05"
-      effort="0"
-      velocity="0" />
-  </joint>
-  <link
-    name="wrist2_Link">
-    <inertial>
-      <origin
-        xyz="-0.00026766 -0.006018 0.051777"
-        rpy="0 0 0" />
-      <mass
-        value="0.47808" />
-      <inertia
-        ixx="0.00043632"
-        ixy="-3.8419E-07"
-        ixz="1.3899E-06"
-        iyy="0.00042788"
-        iyz="3.1286E-05"
-        izz="0.00038517" />
-    </inertial>
-    <visual>
-      <origin
-        xyz="0 0 0"
-        rpy="0 0 0" />
-      <geometry>
-        <mesh
-          filename="package://aubo_description/meshes/aubo_e5/visual/wrist2_Link.DAE" />
-      </geometry>
-      <material
-        name="">
-        <color
-          rgba="1 1 1 1" />
-      </material>
-    </visual>
-    <collision>
-      <origin
-        xyz="0 0 0"
-        rpy="0 0 0" />
-      <geometry>
-        <mesh
-          filename="package://aubo_description/meshes/aubo_e5/collision/wrist2_Link.STL" />
-      </geometry>
-    </collision>
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
Commit message: 快换

File: aubo_ros2_ws/src/aubo_ros2_driver/aubo_description/urdf/xacro/inc/aubo_ros2.xacro (robot description, xacro)
@@ -10,32 +10,4 @@
   <!-- Include GitHub E5_10 URDF (cleaned version) -->
   <xacro:include filename="$(find aubo_description)/urdf/aubo_e5_10_clean.urdf" />
-  <!-- 盒子模型：相对 world，偏移 x=0.4 y=0.18 z=高度一半=0.04，长宽 0.2 高 0.08 -->
-  <link name="box_link">
-    <inertial>
-      <origin xyz="0 0 0" rpy="0 0 0" />
-      <mass value="0.1" />
-      <inertia ixx="0.0001" ixy="0" ixz="0" iyy="0.0001" iyz="0" izz="0.0001" />
-    </inertial>
-    <visual>
-      <origin xyz="0 0 0" rpy="0 0 0" />
-      <geometry>
-        <box size="0.2 0.2 0.08" />
-      </geometry>
-      <material name="box_material">
-        <color rgba="0.6 0.4 0.2 1" />
-      </material>
-    </visual>
-    <collision>
-      <origin xyz="0 0 0" rpy="0 0 0" />
-      <geometry>
-        <box size="0.2 0.2 0.08" />
-      </geometry>
-    </collision>
-  </link>
-  <joint name="world_to_box_joint" type="fixed">
-    <parent link="world" />
-    <child link="box_link" />
-    <origin xyz="0.4 0.18 0.04" rpy="0 0 0" />
-  </joint>
   <!-- MoveIt2 Tool Center Point -->
   <link name="tool_tcp">
@@ -67,5 +39,5 @@
       <origin xyz="0 0 0" rpy="0 0 0" />
       <geometry>
-        <box size="1.5 0.8 0.1" />
+        <box size="1.5 0.6 0.1" />
       </geometry>
       <material name="">
@@ -76,5 +48,5 @@
       <origin xyz="0 0 0" rpy="0 0 0" />
       <geometry>
-        <box size="1.5 0.8 0.1" />
+        <box size="1.5 0.6 0.1" />
       </geometry>
     </collision>

Commit message: 快换测试成功

File: aubo_ros2_ws/src/aubo_ros2_driver/aubo_description/urdf/xacro/inc/aubo_ros2.xacro (robot description, xacro)
@@ -39,5 +39,5 @@
       <origin xyz="0 0 0" rpy="0 0 0" />
       <geometry>
-        <box size="1.5 0.6 0.1" />
+        <box size="1.5 0.5 0.1" />
       </geometry>
       <material name="">
@@ -48,5 +48,5 @@
       <origin xyz="0 0 0" rpy="0 0 0" />
       <geometry>
-        <box size="1.5 0.6 0.1" />
+        <box size="1.5 0.5 0.1" />
       </geometry>
     </collision>

Commit message: chore: 清理调试 instrumentation 并添加夹爪快换 Worker
- 移除 aubo_ros2_trajectory_action、movel_server、aubo_driver_ros2、aubo_robot_simulator 中的 debug 日志写入
- 新增 moveit_arcline_gripper_worker：夹爪快换服务 run_gripper_swap（gripper0_to_gripper2 / gripper2_to_gripper0）
- 新增 RunGripperSwap.srv 服务接口

Made-with: Cursor

File: aubo_ros2_ws/src/aubo_ros2_driver/aubo_description/urdf/xacro/inc/aubo_ros2.xacro (robot description, xacro)
@@ -26,10 +26,5 @@
       </material>
     </visual>
-    <collision>
-      <origin xyz="0 0 0" rpy="0 0 0" />
-      <geometry>
-        <box size="0.2 0.2 0.08" />
-      </geometry>
-    </collision>
+    <!-- no collision geometry for box_link -->
   </link>
   <joint name="world_to_box_joint" type="fixed">
@@ -73,10 +68,5 @@
       </material>
     </visual>
-    <collision>
-      <origin xyz="0 0 0" rpy="0 0 0" />
-      <geometry>
-        <box size="1.5 0.8 0.1" />
-      </geometry>
-    </collision>
+    <!-- no collision geometry for pedestal_Link -->
   </link>
   <joint name="pedestal_joint" type="fixed">

Commit message: 多任务串联仿真完成

File: aubo_ros2_ws/src/aubo_ros2_driver/aubo_description/urdf/xacro/inc/aubo_ros2.xacro (robot description, xacro)
@@ -10,27 +10,4 @@
   <!-- Include E5_10 base URDF (cleaned, in standard robots/) -->
   <xacro:include filename="$(find aubo_description)/urdf/robots/aubo_e5_10_clean.urdf" />
-  <!-- 盒子模型：相对 world，偏移 x=0.4 y=0.18 z=高度一半=0.04，长宽 0.2 高 0.08 -->
-  <link name="box_link">
-    <inertial>
-      <origin xyz="0 0 0" rpy="0 0 0" />
-      <mass value="0.1" />
-      <inertia ixx="0.0001" ixy="0" ixz="0" iyy="0.0001" iyz="0" izz="0.0001" />
-    </inertial>
-    <visual>
-      <origin xyz="0 0 0" rpy="0 0 0" />
-      <geometry>
-        <box size="0.2 0.2 0.08" />
-      </geometry>
-      <material name="box_material">
-        <color rgba="0.6 0.4 0.2 1" />
-      </material>
-    </visual>
-    <!-- no collision geometry for box_link -->
-  </link>
-  <joint name="world_to_box_joint" type="fixed">
-    <parent link="world" />
-    <child link="box_link" />
-    <origin xyz="0.4 0.18 0.04" rpy="0 0 0" />
-  </joint>
   <!-- MoveIt2 Tool Center Point -->
   <link name="tool_tcp">
