Commit message: 机械臂模型web

File: aubo_ros2_ws/src/aubo_ros2_driver/aubo_description/urdf/robots/aubo_robot.urdf (robot description, URDF)
Before this commit: robot aubo_robot, 20 links, 19 joints
Links:
- link camera_Link: geometry collision box size=0.08 0.06 0.05; visual box size=0.08 0.06 0.05
- link grap0_Link: geometry collision box size=0.03 0.06 0.025; visual box size=0.03 0.06 0.025
- link grap1_Link: geometry collision box size=0.03 0.06 0.025; visual box size=0.03 0.06 0.025
- link grap_Link: geometry collision box size=0.10 0.08 0.05; visual box size=0.10 0.08 0.05
- link kuaihuan_Link: geometry collision box size=0.05 0.05 0.03; visual box size=0.05 0.05 0.03

File: aubo_ros2_ws/src/aubo_ros2_driver/aubo_description/urdf/robots/aubo_robot.urdf.xacro (robot description, xacro)
@@ -243,14 +243,14 @@
       <origin rpy="0 0 0" xyz="0 0 0"/>
       <geometry>
-        <mesh filename="package://aubo_description/meshes/end_effector/camera_Link.STL"/>
-      </geometry>
-      <material name="">
-        <color rgba="1 1 1 1"/>
-      </material>
-    </visual>
-    <collision>
-      <origin rpy="0 0 0" xyz="0 0 0"/>
-      <geometry>
-        <mesh filename="package://aubo_description/meshes/end_effector/camera_Link.STL"/>
+        <box size="0.08 0.06 0.05"/>
+      </geometry>
+      <material name="">
+        <color rgba="1 1 1 1"/>
+      </material>
+    </visual>
+    <collision>
+      <origin rpy="0 0 0" xyz="0 0 0"/>
+      <geometry>
+        <box size="0.08 0.06 0.05"/>
       </geometry>
     </collision>
@@ -271,14 +271,14 @@
       <origin rpy="0 0 0" xyz="0 0 0"/>
       <geometry>
-        <mesh filename="package://aubo_description/meshes/end_effector/kuaihuan_Link.STL"/>
-      </geometry>
-      <material name="">
-        <color rgba="1 1 1 1"/>
-      </material>
-    </visual>
-    <collision>
-      <origin rpy="0 0 0" xyz="0 0 0"/>
-      <geometry>
-        <mesh filename="package://aubo_description/meshes/end_effector/kuaihuan_Link.STL"/>
+        <box size="0.05 0.05 0.03"/>
+      </geometry>
+      <material name="">
+        <color rgba="1 1 1 1"/>
+      </material>
+    </visual>
+    <collision>
+      <origin rpy="0 0 0" xyz="0 0 0"/>
+      <geometry>
+        <box size="0.05 0.05 0.03"/>
       </geometry>
     </collision>
@@ -299,5 +299,5 @@
       <origin rpy="0 0 0" xyz="0 0 0"/>
       <geometry>
-        <mesh filename="package://aubo_description/meshes/end_effector/grap_Link.STL"/>
+        <box size="0.10 0.08 0.05"/>
       </geometry>
       <material name="">
@@ -308,5 +308,5 @@
       <origin rpy="0 0 0" xyz="0 0 0"/>
       <geometry>
-        <mesh filename="package://aubo_description/meshes/end_effector/grap_Link.STL"/>
+        <box size="0.10 0.08 0.05"/>
       </geometry>
     </collision>
@@ -327,5 +327,5 @@
       <origin rpy="0 0 0" xyz="0 0 0"/>
       <geometry>
-        <mesh filename="package://aubo_description/meshes/end_effector/grap0_Link.STL"/>
+        <box size="0.03 0.06 0.025"/>
       </geometry>
       <material name="">
@@ -336,5 +336,5 @@
       <origin rpy="0 0 0" xyz="0 0 0"/>
       <geometry>
-        <mesh filename="package://aubo_description/meshes/end_effector/grap0_Link.STL"/>
+        <box size="0.03 0.06 0.025"/>
       </geometry>
     </collision>
@@ -355,5 +355,5 @@
       <origin rpy="0 0 0" xyz="0 0 0"/>
       <geometry>
-        <mesh filename="package://aubo_description/meshes/end_effector/grap1_Link.STL"/>
+        <box size="0.03 0.06 0.025"/>
       </geometry>
       <material name="">
@@ -364,5 +364,5 @@
       <origin rpy="0 0 0" xyz="0 0 0"/>
       <geometry>
-        <mesh filename="package://aubo_description/meshes/end_effector/grap1_Link.STL"/>
+        <box size="0.03 0.06 0.025"/>
       </geometry>
     </collision>

File: aubo_ros2_ws/src/aubo_ros2_driver/aubo_description/urdf/xacro/inc/end_effector.xacro (robot description, xacro)
@@ -1,4 +1,5 @@
 <?xml version="1.0"?>
 <robot xmlns:xacro="http://ros.org/wiki/xacro">
+  <!-- 末端几何使用 package://aubo_description/meshes/end_effector/*.STL（源码见 src/.../meshes/end_effector）。 -->
   <!-- /////////////////////////////////   Camera Link   ////////////////////////////////////// -->
   <link name="camera_Link">
