Commit message: feat: 新旧两套机械臂驱动架构并存 — 新增独立控制器/状态广播器/Dashboard节点
新架构核心: AuboHardwareInterface 封装 SDK 双连接 + JointTrajectoryController
(200Hz C++ 插值) + DashboardNode + StateBroadcaster, 通过 aubo_new_driver.launch.py 启动。
旧架构保留 aubo_driver_ros2 单节点多线程模式, 两套可独立运行。

Co-Authored-By: Claude Opus 4.7 <noreply@anthropic.com>

File: aubo_ros2_ws/src/aubo_ros2_driver/aubo_description/urdf/aubo_e5_10.urdf (robot description, URDF)
Before this commit: robot aubo_e5_10, 14 links, 13 joints
Links:
- link coffee_Link: mass 91.2843777246585 -> 91.454
Joints:
- joint coffee_joint: origin xyz=-0.53995 0.20318 0.016 rpy=1.5708 0 1.5708 -> xyz=-0.53995 0.20318 0.046 rpy=1.5708 0 1.5708

File: aubo_ros2_ws/src/aubo_ros2_driver/aubo_moveit_config/config/aubo_e5.urdf.xacro (robot description, xacro)
@@ -3,6 +3,54 @@
   <xacro:arg name="ros2_control_hardware_type" default="mock_components"/>
   <xacro:arg name="use_fake_hardware" default="true"/>
+  <xacro:arg name="gripper" default=""/>
   <!-- 基础 E5-10 机械臂 URDF（aubo_description，含末端执行器） -->
   <xacro:include filename="$(find aubo_description)/urdf/aubo_e5_10.urdf"/>
+  <!-- ═══════════════════════════════════════════════════════════════ -->
+  <!-- 动态末端：通过 gripper 参数选择挂载到 kuaihuan_Link 的工具  -->
+  <!-- ═══════════════════════════════════════════════════════════════ -->
+  <xacro:macro name="gripper_link" params="name mesh_file">
+    <link name="${name}_Link">
+      <visual>
+        <origin xyz="0 0 0" rpy="0 0 0"/>
+        <geometry>
+          <mesh filename="package://aubo_description/meshes/visual/${mesh_file}"/>
+        </geometry>
+        <material name="${name}_material">
+          <color rgba="0.5 0.5 0.5 1.0"/>
+        </material>
+      </visual>
+      <collision>
+        <origin xyz="0 0 0" rpy="0 0 0"/>
+        <geometry>
+          <mesh filename="package://aubo_description/meshes/collision/${mesh_file}"/>
+        </geometry>
+      </collision>
+    </link>
+    <joint name="kuaihuan_to_${name}" type="fixed">
+      <parent link="kuaihuan_Link"/>
+      <child link="${name}_Link"/>
+      <origin xyz="0 0 0.033" rpy="0 0 0"/>
+    </joint>
+  </xacro:macro>
+  <!-- gripper0: 气动夹爪 φ40 -->
+  <xacro:if value="${'$(arg gripper)' == 'gripper0'}">
+    <xacro:gripper_link name="gripper0" mesh_file="gripper0_link.stl"/>
+  </xacro:if>
+  <!-- gripper1: 电动夹爪 A -->
+  <xacro:if value="${'$(arg gripper)' == 'gripper1'}">
+    <xacro:gripper_link name="gripper1" mesh_file="gripper1_link.stl"/>
+  </xacro:if>
+  <!-- gripper2: 电动夹爪 φ60 -->
+  <xacro:if value="${'$(arg gripper)' == 'gripper2'}">
+    <xacro:gripper_link name="gripper2" mesh_file="gripper2_link.stl"/>
+  </xacro:if>
+  <!-- gripper1coffeecup: 咖啡杯工具 -->
+  <xacro:if value="${'$(arg gripper)' == 'gripper1coffeecup'}">
+    <xacro:gripper_link name="gripper1coffeecup" mesh_file="gripper1coffeecup_link.stl"/>
+  </xacro:if>
+  <!-- gripper1milkcup: 牛奶杯工具 -->
+  <xacro:if value="${'$(arg gripper)' == 'gripper1milkcup'}">
+    <xacro:gripper_link name="gripper1milkcup" mesh_file="gripper1milkcup_link.stl"/>
+  </xacro:if>
   <!-- Tool Center Point -->
   <link name="tool_tcp">

Commit message: feat: RViz2 动态 URDF 重载 + 平滑渲染夹爪 + 去掉 AttachedCollisionObject
核心改动:
- moveit_ros_visualization: PlanningSceneDisplay 订阅 /robot_description 话题动态重载 RobotModel
- moveit_ros_planning_interface: 新增 clearSharedRobotModelLoader() 清除静态缓存
- tool_changer: scene_attach_worker 直接发布 URDF 到 /robot_description 话题
- tool_changer: 去掉冗余 AttachedCollisionObject，改用 URDF 碰撞几何 + Assimp 平滑渲染
- 文档: ARCHITECTURE.md 新增动态 URDF 重载章节

调试修复:
- fix: 删除未实现的 publishToolMarker() 和 visualization_msgs include
- fix: onRobotDescriptionTopic 首次消息跳过 + declare_parameter 防止崩溃
- fix: createPlanningSceneMonitor 直接构造 RobotModelLoader(Options(urdf, srdf))
  绕过 getSharedRobotModelLoader 静态缓存（overlay/underlay SharedStorage 独立副本问题）
- fix: source 顺序 overlay 最后保证 include 路径优先

Co-Authored-By: Claude Opus 4.7 <noreply@anthropic.com>

File: aubo_ros2_ws/src/aubo_ros2_driver/aubo_description/urdf/aubo_e5_10.urdf (robot description, URDF)
Before this commit: robot aubo_e5_10, 14 links, 13 joints
Joints:
- removed joint base_joint
- added joint world_to_base: type fixed, parent world, child base_link, origin xyz=0.0 0.0 0.0 rpy=0 0 0
- joint world_to_pedestal: origin xyz=0.0 0.0 0.0 rpy=0.0 0.0 0.0 -> xyz=-0.10483 -0.10483 -0.028 rpy=0.0 0.0 0.0

File: aubo_ros2_ws/src/aubo_ros2_driver/aubo_moveit_config/config/aubo_e5.urdf.xacro (robot description, xacro)
@@ -9,5 +9,16 @@
   <!-- 动态末端：通过 gripper 参数选择挂载到 kuaihuan_Link 的工具  -->
   <!-- ═══════════════════════════════════════════════════════════════ -->
-  <xacro:macro name="gripper_link" params="name mesh_file">
+  <!--
+    gripper_link 宏: 在 kuaihuan_Link 下挂载末端工具。
+    origin 必须与 tools.yaml 中 attach_offset 一致:
+      gripper0/1:                   pos(0,0,0.033) rpy(0,0,0)
+      gripper2 (z=0.7071,w=0.7071): pos(0,0,0.033) rpy(0,0,π/2) → 90° z
+      gripper1coffeecup (z=1,w=0):  pos(0,0,0.033) rpy(0,0,π)    → 180° z
+      gripper1milkcup (z=-.7071,.7071): pos(0,0,0.033) rpy(0,0,-π/2) → -90° z
+  -->
+  <xacro:macro name="gripper_link"
+               params="name mesh_file
+                       ox:=0 oy:=0 oz:=0.033
+                       rr:=0 rp:=0 ry:=0">
     <link name="${name}_Link">
       <visual>
@@ -30,26 +41,24 @@
       <parent link="kuaihuan_Link"/>
       <child link="${name}_Link"/>
-      <origin xyz="0 0 0.033" rpy="0 0 0"/>
+      <origin xyz="${ox} ${oy} ${oz}" rpy="${rr} ${rp} ${ry}"/>
     </joint>
   </xacro:macro>
-  <!-- gripper0: 气动夹爪 φ40 -->
   <xacro:if value="${'$(arg gripper)' == 'gripper0'}">
     <xacro:gripper_link name="gripper0" mesh_file="gripper0_link.stl"/>
   </xacro:if>
-  <!-- gripper1: 电动夹爪 A -->
   <xacro:if value="${'$(arg gripper)' == 'gripper1'}">
     <xacro:gripper_link name="gripper1" mesh_file="gripper1_link.stl"/>
   </xacro:if>
-  <!-- gripper2: 电动夹爪 φ60 -->
   <xacro:if value="${'$(arg gripper)' == 'gripper2'}">
-    <xacro:gripper_link name="gripper2" mesh_file="gripper2_link.stl"/>
+    <xacro:gripper_link name="gripper2" mesh_file="gripper2_link.stl"
+                        ry="${pi/2}"/>
   </xacro:if>
-  <!-- gripper1coffeecup: 咖啡杯工具 -->
   <xacro:if value="${'$(arg gripper)' == 'gripper1coffeecup'}">
-    <xacro:gripper_link name="gripper1coffeecup" mesh_file="gripper1coffeecup_link.stl"/>
+    <xacro:gripper_link name="gripper1coffeecup" mesh_file="gripper1coffeecup_link.stl"
+                        ry="${pi}"/>
   </xacro:if>
-  <!-- gripper1milkcup: 牛奶杯工具 -->
   <xacro:if value="${'$(arg gripper)' == 'gripper1milkcup'}">
-    <xacro:gripper_link name="gripper1milkcup" mesh_file="gripper1milkcup_link.stl"/>
+    <xacro:gripper_link name="gripper1milkcup" mesh_file="gripper1milkcup_link.stl"
+                        ry="${-pi/2}"/>
   </xacro:if>
   <!-- Tool Center Point -->
