Commit message: v1

File: aubo_ros2_ws/src/aubo_ros2_driver/aubo_description/urdf/aubo_e5_10.urdf (robot description, URDF)
Before this commit: robot aubo_e5_10, 8 links, 7 joints
Links:
- added link box_link, mass 0.1; collision box size=0.2 0.2 0.08; visual box size=0.2 0.2 0.08
Joints:
- added joint world_to_box_joint: type fixed, parent world, child box_link, origin xyz=0.4 0.18 0.04 rpy=0 0 0

File: aubo_ros2_ws/src/aubo_ros2_driver/aubo_description/urdf/xacro/inc/aubo_ros2.xacro (robot description, xacro)
@@ -10,4 +10,32 @@
   <!-- Include GitHub E5_10 URDF (cleaned version) -->
   <xacro:include filename="$(find aubo_description)/urdf/aubo_e5_10_clean.urdf" />
+  <!-- 盒子模型：相对 world，偏移 x=0.4 y=0.18 z=高度一半=0.04，长宽 0.2 高 0.08 -->
+  <link name="box_link">
+    <inertial>
+      <origin xyz="0 0 0" rpy="0 0 0" />
+      <mass value="0.1" />
+      <inertia ixx="0.0001" ixy="0" ixz="0" iyy="0.0001" iyz="0" izz="0.0001" />
+    </inertial>
+    <visual>
+      <origin xyz="0 0 0" rpy="0 0 0" />
+      <geometry>
+        <box size="0.2 0.2 0.08" />
+      </geometry>
+      <material name="box_material">
+        <color rgba="0.6 0.4 0.2 1" />
+      </material>
+    </visual>
+    <collision>
+      <origin xyz="0 0 0" rpy="0 0 0" />
+      <geometry>
+        <box size="0.2 0.2 0.08" />
+      </geometry>
+    </collision>
+  </link>
+  <joint name="world_to_box_joint" type="fixed">
+    <parent link="world" />
+    <child link="box_link" />
+    <origin xyz="0.4 0.18 0.04" rpy="0 0 0" />
+  </joint>
   <!-- MoveIt2 Tool Center Point -->
   <link name="tool_tcp">
@@ -57,5 +85,6 @@
     <origin xyz="0.0 0.0 -0.05" rpy="0.0 0.0 0.0" />
   </joint>
-  <!-- pedestal square link (optional table) -->
+  <!-- pedestal square link (optional table) - temporarily commented -->
+  <!--
   <link name="pedestal_square_link">
     <inertial>
@@ -85,4 +114,5 @@
     <origin xyz="-0.55 0.0 0.16" rpy="0.0 0.0 0.0" />
   </joint>
+  -->
   <!-- gazebo color -->
   <gazebo reference="pedestal_Link">

File: aubo_ros2_ws/src/aubo_ros2_driver/aubo_description/urdf/xacro/inc/end_effector.xacro (robot description, xacro)
@@ -280,7 +280,7 @@
   </link>
   <joint name="grap1_to_tip_joint" type="fixed">
-    <parent link="grap1_Link" />
+    <parent link="wrist3_Link" />
     <child link="gripper_tip_link" />
-    <origin xyz="-0.01 0.047 0.0" rpy="0.0 0.0 0.0" />
+    <origin xyz="0.0 0.0 0.185" rpy="0.0 0.0 0.0" />
   </joint>
 </robot>

Commit message: 机械臂取拿牛奶杯测试轨迹

File: aubo_ros2_ws/src/aubo_ros2_driver/aubo_description/urdf/aubo_e5_10.urdf (robot description, URDF)
Before this commit: robot aubo_e5_10, 14 links, 13 joints
Links:
- removed link lizhu_Link
Joints:
- removed joint lizhu_joint

Commit message: “机械臂牛奶杯示教完成”

File: aubo_ros2_ws/src/aubo_ros2_driver/aubo_description/urdf/aubo_e5_10.urdf (robot description, URDF)
Before this commit: robot aubo_e5_10, 13 links, 12 joints
Links:
- added link lizhu_Link, mass 0.86598; collision mesh filename=package://aubo_description/meshes/collision/lizhu_link.stl; visual mesh filename=package://aubo_description/meshes/visual/lizhu_link.stl
Joints:
- added joint lizhu_joint: type fixed, parent pedestal_Link, child lizhu_Link, origin xyz=-0.630 -0.3675 0.006 rpy=1.5708 0 1.5708

Commit message: “6月2日拉花失败版本，但是优化graspnet”

File: aubo_ros2_ws/src/aubo_ros2_driver/aubo_description/urdf/aubo_e5_10.urdf (robot description, URDF)
Before this commit: robot aubo_e5_10, 13 links, 12 joints
Links:
- added link lizhu_Link, mass 0.86598; collision mesh filename=package://aubo_description/meshes/collision/lizhu_link.stl; visual mesh filename=package://aubo_description/meshes/visual/lizhu_link.stl
- added link paper_cup_Link, mass 0.01; collision mesh filename=package://aubo_description/meshes/collision/paper_cup.stl; visual mesh filename=package://aubo_description/meshes/visual/paper_cup.stl
Joints:
- added joint lizhu_joint: type fixed, parent pedestal_Link, child lizhu_Link, origin xyz=-0.630 -0.3675 0.006 rpy=1.5708 0 1.5708
- added joint paper_cup_joint: type fixed, parent pedestal_Link, child paper_cup_Link, origin xyz=-0.630 -0.3075 0.106 rpy=0 0 0

File: aubo_ros2_ws/src/aubo_ros2_driver/aubo_moveit_config/config/aubo_e5.urdf.xacro (robot description, xacro)
@@ -62,5 +62,5 @@
                         ry="${-pi/2}"/>
   </xacro:if>
-  <!-- Tool Center Point -->
+  <!-- Tool Center Point (红色, r=5mm) -->
   <link name="tool_tcp">
     <visual>
@@ -78,4 +78,11 @@
     <child link="tool_tcp"/>
     <origin xyz="0.0 0.0 0.0235" rpy="0.0 0.0 0.0"/>
+  </joint>
+  <!-- 奶缸嘴 (spout tip) — 末端工具坐标系, 标定值: TCP→spout = (-38,95,212)mm 喵~ -->
+  <link name="spout_marker"/>
+  <joint name="tcp_to_spout" type="fixed">
+    <parent link="tool_tcp"/>
+    <child link="spout_marker"/>
+    <origin xyz="-0.038 0.095 0.212" rpy="0 0 0"/>
   </joint>
   <!-- Transmission -->
