Commit message: 采摘链路代码优化（2026-08-14 19:20，代码优化未测试）
- 安全门分层：目标身份/新鲜度判定上移 BT 层单点决策，运动层与 MTC
  执行边界只留硬件安全门 safetyReady（修复真机 stale 致死根因：
  BT 放行策略被内层门互相否决）
- 抓取端：goal 目标钉死（受理与 Prepare 间 selected 切换即失败重派）、
  waitForRefined 谓词以位姿到达为准（fitting 单独到达不再绕过降级链）、
  降级行程 suggested 无效时取量程中点、post-set 回调改参全量生效、
  质量门/视点规划结构体默认值对齐 yaml、观察段时间盒 scan.time_budget_s=5.0
  （暂时测试设置）、拒绝日志带原因
- 感知端：推理 worker 异常保护（异常不再杀线程静默无输出）、YOLO detect
  保护、SAM 批量分割一次调用、记忆锚点 entry_pose 回填、masks 保存每目标
  节流 1s、删除 segment_detections 死代码
- 编排端：熔断阈值参数化 dispatch.max_consecutive_rejections=6、38 条
  枚举↔消息常量 static_assert 编译期护栏、batch_completed 事件去重、
  README 语义对齐
- 新增整体设计文档 docs/superpowers/specs/2026-08-14-peach-harvest-integral-design.md
  （分层架构/状态机/接口契约/安全门分层/Refinement Journal 设计/问题登记册）

状态：编译通过（peach_approach_grasp/peach_harvest_orchestrator 等），
今日未跑 colcon test 与真机验证，代码优化未测试。

File: src/aubo_description/urdf/components/table.xacro (robot description, xacro)
@@ -26,5 +26,8 @@
       <parent link="${parent}"/>
       <child link="table_link"/>
-      <origin xyz="-0.10483 -0.10483 -0.028" rpy="0 0 0"/>
+      <!-- 桌面板上表面（网格系 z=+0.0075）落到世界系 -0.001m：与真机底座
+           所压的真实桌面（=底座底面 z≈-0.0005）贴合，留 0.5mm 防底座与桌面
+           常碰。旧值 -0.028 让模型桌面比真实低 2cm，碰撞检查失真曾致撞桌。 -->
+      <origin xyz="-0.10483 -0.10483 -0.0085" rpy="0 0 0"/>
     </joint>
   </xacro:macro>
