Commit message: feat(peach_sim) 感知验证矩阵轮 M0-M3（852 帧首轮 GATE PASS+基线冻结）+ aubo_description 连接处网格伴随更新
peach_sim reconstruction（PLAN.md 四里程碑全落地）：
- M0 红项收口：add_bag 生成期 BVH 间隙校验（果球按需收缩至 ≥0.5mm，fruit_clearance_m 逐袋入 manifest）几何门 0 errors；Cycles 切 OptiX（RTX 3090，三机位 48samples 40.7s）；perception_validation.json+reference_depth_mm.png 落盘，深度对照 9 袋 MAE 13.5mm
- M1 blender_orchard 并入删除：measure_priors/make_textures 迁入（贴图 sha256 逐字节一致）；crease warp 0.005 并入 geometry；paper.png 裁定 bump-only（颜色乘法 recall 9→7，回退后 9/9 恢复）；git rm blender_orchard/ 全仓引用清理
- M2 条件参数化：lighting.py 四光照预设（Nishita Air/Dust 映射浑浊度）；occlusion.py 名义档+heavy 横枝+走廊枝（对齐 L_insert 0.090）；袋宽高按 priors 分位逆采样逐袋 source_percentile 入 manifest；--scale validation|field（field=3行×8株393袋锚定场）
- M3 多视角矩阵：viewpoints.py 停走停靠+补视复刻 view_policy（1e-9 对拍双实现防漂移）；852 帧=4 光照×69 目标×3 视序列+6 停靠，24samples OptiX 57min 独占；评测分层：覆盖率桶单调（low .59/mid .28/high .03）、袋级 any_view none .825/light .775/heavy .537/参考 .944、overcast 全档低 8-15%；裁定评测主分层=深度反测覆盖率桶（名义遮挡档被自然本底淹没倒挂）
- 基线冻结 baselines/perception_matrix_baseline.json（容差 0.05，--gate 复验 PASS）；帧本体 8.1G gitignore 可重现、摘要 matrix_*.{json,md} 入库；test_reconstruction_core.py 19 测全绿；lint 债归属核实记档（I100/I201 存量，留专项轮）；坑：双 Blender 并发抢 3090 OOM 须串行
- 文档同轮：peach_sim README 单入口重写、PLAN/RESULTS 追加、architecture/io/testing 三活文档更新、testing-log 两节；field_anchor 535M 渲染帧补 gitignore（--scale field 可重现）

aubo_description（09-28 连接处重叠审计后续）：camera_bracket.stl 双档相机支架网格、quick_changer_adaptive.stl 专用快换、render_joint_check.py 连接处渲染检查脚本；camera/quick_changer/tcp 系 xacro 与三剪切工具网格同步更新

File: src/aubo_description/urdf/components/camera.xacro (robot description, xacro)
@@ -23,9 +23,28 @@
         </geometry>
       </collision>
+      <!-- 2026-09-28 补托架：本版 STEP「相机安装板」为空组（FreeCAD 提不出），
+           几何取自 ros2_qws 同源逐件导出（自适应总装 相机安装板2，wrist3 系建模）。
+           安装板随工具总装而异（咬合装=安装板1 y[-31,90]），单资产先随默认 adaptive。 -->
+      <visual>
+        <geometry>
+          <mesh filename="package://aubo_description/meshes/visual/sensors/camera_bracket.stl"/>
+        </geometry>
+        <material name="camera_gray">
+          <color rgba="0.82 0.82 0.82 1.0"/>
+        </material>
+      </visual>
+      <collision>
+        <geometry>
+          <mesh filename="package://aubo_description/meshes/collision/sensors/camera_bracket.stl"/>
+        </geometry>
+      </collision>
     </link>
     <joint name="camera_mount_joint" type="fixed">
       <parent link="${parent}"/>
       <child link="camera_body_link"/>
-      <origin xyz="0 0 0.020" rpy="0 0 0"/>
+      <!-- 2026-09-28：网格自 STEP 总装重提（PS800-E1相机005，y[90,137] z[-50,20]mm，
+           wrist3 系建模；该版 STEP 相机安装板为空组未建托架），原点随网格系归零。
+           手眼外参链锚 wrist3_Link→camera_link 不经本帧，位姿变更零影响。 -->
+      <origin xyz="0 0 0" rpy="0 0 0"/>
     </joint>
   </xacro:macro>

File: src/aubo_description/urdf/components/quick_changer.xacro (robot description, xacro)
@@ -1,4 +1,6 @@
 <?xml version="1.0"?>
 <robot xmlns:xacro="http://www.ros.org/wiki/xacro">
+  <!-- 2026-09-28 起本链接保留为帧（名冻结：SRDF/ACM/octomap 豁免名单按名消费），不再挂几何——
+       快换盘对与等高垫块已并入各 profile 的 tool_body_link（一次导出方式，见 tcp.xacro）。 -->
   <xacro:macro name="aubo_e5_quick_changer" params="parent:=camera_body_link">
     <link name="quick_changer_link">
@@ -7,24 +9,11 @@
         <mass value="0.21939"/>
         <inertia ixx="6.3771e-05" ixy="4.2875e-07" ixz="-1.7848e-07"
-                 iyy="6.9403e-05" iyz="-4.5085e-07" izz="0.0001149"/>
+                 iyy="6.9400e-05" iyz="-4.5085e-07" izz="0.0001149"/>
       </inertial>
-      <visual>
-        <geometry>
-          <mesh filename="package://aubo_description/meshes/visual/tools/quick_changer.stl"/>
-        </geometry>
-        <material name="quick_changer_gray">
-          <color rgba="0.82 0.82 0.82 1.0"/>
-        </material>
-      </visual>
-      <collision>
-        <geometry>
-          <mesh filename="package://aubo_description/meshes/collision/tools/quick_changer.stl"/>
-        </geometry>
-      </collision>
     </link>
     <joint name="quick_changer_mount_joint" type="fixed">
       <parent link="${parent}"/>
       <child link="quick_changer_link"/>
-      <origin xyz="0 0 0.0215" rpy="0 0 3.1416"/>
+      <origin xyz="0 0 0" rpy="0 0 0"/>
     </joint>
   </xacro:macro>

File: src/aubo_description/urdf/components/tcp.xacro (robot description, xacro)
@@ -3,5 +3,5 @@
   <!-- 末端 TCP 共享底座：帧名冻结（tool_axis/cutting_plane/tcp/sleeve_mouth/tool_body_link），
        SRDF 链 tip、ACM×octomap 豁免名单、技能/重建的三点 TF 验证均按名消费，不得改名。
-       2026-09-28 起三把剪切手共用（shear_v1 / bite_shear_v1 / adaptive_shear_v1，替换两把套袋圆柱）：
+       2026-09-28 起三把剪切手共用（shear_v1 / bite_shear_v1 / adaptive_shear_v1）：
        tool_axis 原点/姿态、sleeve_mouth 偏移、网格名由各 wrapper（tcp_<profile>.xacro）传入；
        几何档案：aubo_description/config/<profile>.yaml（改几何改 wrapper 与档案两处）。
@@ -9,8 +9,12 @@
        cutting_plane / tcp 与 tool_axis 同点（刀口深度登记在档案 geometry_m.L_blade）。
        tool_body_link 直接挂 parent：网格在法兰系（=parent 系）下建模，identity 落位；
-       CAD 原点 = wrist3_Link 原点已数值验证（link6 Ø75 法兰 + STW 快换盘 + 相机族三方叠对）。
+       CAD 原点 = wrist3_Link 原点已数值验证（link6 Ø75 法兰叠对，ros2_qws ICP 复核）。
+       2026-09-28 一次导出方式（ros2_qws 同构）：tool_body_link 同时承载本 profile 总装的
+       快换盘对（changer_stem）与等高垫块圆柱（spacer_len）——每工具栈自洽无跨装配错位；
+       法兰-主盘间隙的垫块未建模（全部 STEP 同），以圆柱代理，真机测绘后替换。
+       quick_changer_link / camera_body_link 保留为帧（名冻结），几何已并入本链接与相机链接。
        STEP→网格管线：scripts/step_extract_tool.py + scripts/decimate_export.py。
        不得再用 static_transform_publisher 补发 wrist3_Link→tcp。 -->
-  <xacro:macro name="aubo_e5_tcp" params="parent:=wrist3_Link tcp_xyz:='0 0 0' tcp_rpy:='-1.5708 0 0' sleeve_mouth_z:=0.0 mesh_stem:=shear_v1 body_rgba:='0.55 0.58 0.62 1.0'">
+  <xacro:macro name="aubo_e5_tcp" params="parent:=wrist3_Link tcp_xyz:='0 0 0' tcp_rpy:='-1.5708 0 0' sleeve_mouth_z:=0.0 mesh_stem:=shear_v1 body_rgba:='0.55 0.58 0.62 1.0' changer_stem:='quick_changer' spacer_len:=0.0147">
     <link name="tool_axis"/>
     <joint name="tool_axis_joint" type="fixed">
@@ -38,5 +42,5 @@
     </joint>
     <link name="tool_body_link">
-      <!-- 网格在法兰系（parent 系）下建模：identity 挂 parent 即正确落位 -->
+      <!-- 工具网格（法兰系建模，identity 落位） -->
       <visual>
         <geometry>
@@ -52,4 +56,34 @@
         </geometry>
       </collision>
+      <!-- 本 profile 总装的 STW 主盘+付盘锁定对（z 上沿=该装配付盘顶） -->
+      <visual>
+        <geometry>
+          <mesh filename="package://aubo_description/meshes/visual/tools/${changer_stem}.stl"/>
+        </geometry>
+        <material name="tool_body_mat">
+          <color rgba="${body_rgba}"/>
+        </material>
+      </visual>
+      <collision>
+        <geometry>
+          <mesh filename="package://aubo_description/meshes/collision/tools/${changer_stem}.stl"/>
+        </geometry>
+      </collision>
+      <!-- 法兰→主盘底等高垫块（CAD 未建模，圆柱代理） -->
+      <visual>
+        <origin xyz="0 0 ${spacer_len / 2}" rpy="0 0 0"/>
+        <geometry>
+          <cylinder radius="0.0495" length="${spacer_len}"/>
+        </geometry>
+        <material name="tool_body_mat">
+          <color rgba="${body_rgba}"/>
+        </material>
+      </visual>
+      <collision>
+        <origin xyz="0 0 ${spacer_len / 2}" rpy="0 0 0"/>
+        <geometry>
+          <cylinder radius="0.0495" length="${spacer_len}"/>
+        </geometry>
+      </collision>
     </link>
     <joint name="tool_body_joint" type="fixed">

File: src/aubo_description/urdf/components/tcp_adaptive_shear_v1.xacro (robot description, xacro)
@@ -2,5 +2,5 @@
 <robot xmlns:xacro="http://www.ros.org/wiki/xacro">
   <!-- 自适应剪切手（adaptive_shear_v1，桃子采摘末端执行器）包装：Ø136 圆盘+拉钩组+MPU6050
-       被动自适应贴果；TCP=采摘手外壳工作口圆心 (0, 47, 168.66) mm（总装系测量核定：
+       被动自适应贴果；TCP=采摘手外壳工作口圆心 (0, 47, 168.66) mm（总装测量核定：
        ΔY 47.00 / ΔZ 168.66 / 中心距 175.09，2026-09-28 用户核定）——设计基准与旧
        adaptive_cylinder_v1 完全一致，感知/预抓取/手眼标定链几何零漂移；开口 +Y（Rx(−90°) 传承）。
@@ -10,7 +10,10 @@
   <xacro:include filename="tcp.xacro"/>
   <xacro:macro name="aubo_e5_tcp_adaptive_shear_v1" params="parent:=wrist3_Link">
+    <!-- changer_stem/spacer_len：自适应总装自己的盘对（主盘 [6.7,54.3]/付盘顶 54.5，2026-09-28）；
+         该装配快换栈整体比 shear/bite 两装低 8mm，属 STEP 原装——一次导出方式下各栈自洽。 -->
     <xacro:aubo_e5_tcp parent="${parent}"
         tcp_xyz="0 0.047 0.16866" tcp_rpy="-1.5708 0 0"
         sleeve_mouth_z="0.0" mesh_stem="adaptive_shear_v1"
+        changer_stem="quick_changer_adaptive" spacer_len="0.0067"
         body_rgba="0.60 0.62 0.66 1.0"/>
   </xacro:macro>

File: src/aubo_description/urdf/components/tcp_shear_v1.xacro (robot description, xacro)
@@ -2,10 +2,11 @@
 <robot xmlns:xacro="http://www.ros.org/wiki/xacro">
   <!-- 剪切手（shear_v1，桃子采摘手-相机位置试验版本）包装：连杆切刀在法兰 +Y 侧，
-       开口朝 +Y（Rx(-90°)，与旧套袋圆柱同向）。TCP=连杆切刀对切区中点（CAD preliminary）。
+       开口朝 +Y（Rx(−90°)，与旧套袋圆柱同向）。TCP=传承旧 hollow_cylinder_v1 基准
+       (0, 47.90, 151.07) mm（git 历史核定，2026-09-28 用户裁定）。
        档案：config/shear_v1.yaml；网格 meshes/{visual,collision}/tools/shear_v1.stl。 -->
   <xacro:include filename="tcp.xacro"/>
   <xacro:macro name="aubo_e5_tcp_shear_v1" params="parent:=wrist3_Link">
     <xacro:aubo_e5_tcp parent="${parent}"
-        tcp_xyz="-0.0265 0.053 0.176" tcp_rpy="-1.5708 0 0"
+        tcp_xyz="0 0.0479 0.15107" tcp_rpy="-1.5708 0 0"
         sleeve_mouth_z="0.0" mesh_stem="shear_v1"
         body_rgba="0.55 0.58 0.62 1.0"/>
