Commit message: feat(peach): 双末端工具档案化 adaptive_cylinder_v1 + imu_follow 插入跟随（决策 0020）
- aubo_description：tcp.xacro 参数化为共享底座 + 双 wrapper
  （hollow_cylinder_v1 TCP (0,47.90,151.07)mm / adaptive_cylinder_v1
  TCP (0,47,168.66)mm、D_inner 0.116，帧名共用冻结）；主 xacro 增
  tool_profile arg（默认 adaptive，两个独立 if，未知名缺 tcp 帧即崩）；
  新档案 config/adaptive_cylinder_v1.yaml。固定圆柱展开等价门 diff=0。
- 档案单一事实源：peach_perception/tool_profiles.py launch 期装载注入
  感知 tool.D_inner、重建 tool.budget.d_inner（GraspDecision 许可数学
  随档案）与各包 tool.profile_id 标签；6 处硬编码 hollow 字符串提参。
- launch 穿透：harvest_system/bringup（授权最小穿透）/moveit/
  技能/感知/executor/imu_follow_servo 同 arg 贯穿 RSP 与
  MoveItConfigsBuilder 双展开；ToolProfileValue 替换对象 fail-fast。
- params 新键（模块与 yaml 双改）：tool.profile_id ×3、
  tool.budget.d_inner；重建/场景校验器升级为逐段下钻支持嵌套组。
- imu_follow：新增 ~/insert_start|insert_stop 插入推进（沿工具开口
  低速 0.01 m/s、行程钳 0.20 m、姿态照常跟 IMU）+ insert.* 参数与
  纯核；修 disable 后 IK/goal 回执补发两 bug。
- Web 镜像 to_grasp_decision 增 tool_profile_id；文档同步
  architecture/io/testing + AGENTS 纯核清单 + 三 README。
- 验证：colcon test 116/116；mock 冒烟双向（默认 adaptive：
  全节点标签/内径 0.116、RSP 与 move_group URDF 均含 0.16866、
  生命周期就绪、Web 在线；显式 hollow：0.104/0.15107 同过）。

File: src/aubo_description/urdf/aubo_e5.urdf.xacro (robot description, xacro)
@@ -6,5 +6,6 @@
   <xacro:include filename="components/camera.xacro"/>
   <xacro:include filename="components/quick_changer.xacro"/>
-  <xacro:include filename="components/tcp.xacro"/>
+  <xacro:include filename="components/tcp_hollow_cylinder_v1.xacro"/>
+  <xacro:include filename="components/tcp_adaptive_cylinder_v1.xacro"/>
   <xacro:include filename="aubo_e5.ros2_control.xacro"/>
   <xacro:arg name="include_table" default="true"/>
@@ -14,4 +15,8 @@
   <xacro:arg name="hardware_mode" default="mock"/>
   <xacro:arg name="robot_ip" default="169.254.10.98"/>
+  <!-- tool_profile: hollow_cylinder_v1 (固定圆柱) | adaptive_cylinder_v1 (自适应圆柱+IMU)。
+       两个独立 if（非 if/else）：未知 profile 名两支都不展开 → 缺 tcp 帧，启动即失败。 -->
+  <xacro:arg name="tool_profile" default="adaptive_cylinder_v1"/>
+  <xacro:property name="tool_profile" value="$(arg tool_profile)"/>
   <xacro:aubo_e5_ros2_control
     name="AuboE5System"
@@ -27,5 +32,11 @@
     </xacro:if>
   </xacro:if>
-  <!-- 末端 TCP 固定关节（URDF 内建，robot_state_publisher 发布，见 components/tcp.xacro） -->
-  <xacro:aubo_e5_tcp parent="wrist3_Link"/>
+  <!-- 末端 TCP 固定关节（URDF 内建，robot_state_publisher 发布，见 components/tcp_<profile>.xacro；
+       帧名冻结，两把工具仅 tool_axis 原点不同） -->
+  <xacro:if value="${tool_profile == 'hollow_cylinder_v1'}">
+    <xacro:aubo_e5_tcp_hollow_cylinder_v1 parent="wrist3_Link"/>
+  </xacro:if>
+  <xacro:if value="${tool_profile == 'adaptive_cylinder_v1'}">
+    <xacro:aubo_e5_tcp_adaptive_cylinder_v1 parent="wrist3_Link"/>
+  </xacro:if>
 </robot>

File: src/aubo_description/urdf/components/tcp.xacro (robot description, xacro)
@@ -1,18 +1,19 @@
 <?xml version="1.0"?>
 <robot xmlns:xacro="http://www.ros.org/wiki/xacro">
-  <!-- hollow_cylinder_v1：TCP 在圆柱顶部（开口）。
-       原点机械尺寸 (x=0, y=47.90mm, z=151.07mm) in wrist3_Link。
+  <!-- 末端 TCP 共享底座：帧名冻结（tool_axis/cutting_plane/tcp/sleeve_mouth/tool_body_link），
+       SRDF 链 tip、ACM×octomap 豁免名单、技能/重建的三点 TF 验证均按名消费，不得改名。
+       两把工具仅 tool_axis 原点不同，常量由各 wrapper（tcp_<profile>.xacro）持有；
+       几何档案：aubo_description/config/<profile>.yaml（改几何改 wrapper 与档案两处）。
        TCP 姿态：Z = 开口方向，XY = 刀口平面（剪切在该水平面上）。
        相对法兰 Rx(-90°)，零位开口朝世界 +Z。
        L_blade=0 → cutting_plane / tcp / sleeve_mouth 同点（顶部）；
        筒体沿 TCP −Z 长 L_insert=200mm。
-       不得再用 static_transform_publisher 补发 wrist3_Link→tcp。
-       几何档案：aubo_description/config/hollow_cylinder_v1.yaml -->
-  <xacro:macro name="aubo_e5_tcp" params="parent:=wrist3_Link">
+       不得再用 static_transform_publisher 补发 wrist3_Link→tcp。 -->
+  <xacro:macro name="aubo_e5_tcp" params="parent:=wrist3_Link tcp_xyz:='0 0.0479 0.15107'">
     <link name="tool_axis"/>
     <joint name="tool_axis_joint" type="fixed">
       <parent link="${parent}"/>
       <child link="tool_axis"/>
-      <origin xyz="0 0.0479 0.15107" rpy="-1.5708 0 0"/>
+      <origin xyz="${tcp_xyz}" rpy="-1.5708 0 0"/>
     </joint>
     <link name="cutting_plane"/>

Commit message: feat(s5) 三把剪切手 STEP→URDF 接入（决策 0033）：shear_v1/bite_shear_v1/adaptive_shear_v1 替换两把套袋圆柱。FreeCAD 1.1 snap+Blender 4.5 无头管线入库 aubo_description/scripts/（总装提取/减面/叠对渲染），法兰系=CAD 全局系（link6 Ø75+STW 快换+相机族三方数值叠对+三工具渲染叠图双验收）；网格双档 5.5万/4.5k tri 入 meshes/tools/；tcp.xacro 参数化（帧名冻结/SRDF 零改/tool_body_link 挂 parent），档案 preliminary_cad（TCP/张口/包络 CAD 推导待真机标定）；注入面扩 body_length/body_radius 随档案；bringup tool_profile 去 choices 纯透传；usesImuFollowContact/imu_follow 条件→adaptive_shear_v1、insert.max_travel 0.09 对齐档案；peach_sim 镜像+世界重生成；xacro×3+check_urdf/colcon build 10 包/peach_harvester 219 测/冒烟三 profile TF 数值对档案全过；记档：E1 C03 转红=注入器 known-good 目标随工具几何失配待 E1 轮重标、exit -6=先在 F-E1-1、r0_gate manifest 红=先在 c53b177；坑：CMake 3.28 下 _FOUND TRUE 短路失效须 AMENT_LINT_AUTO_EXCLUDE、Blender 无头渲染须 camera_add 管线

File: src/aubo_description/urdf/aubo_e5.urdf.xacro (robot description, xacro)
@@ -6,6 +6,7 @@
   <xacro:include filename="components/camera.xacro"/>
   <xacro:include filename="components/quick_changer.xacro"/>
-  <xacro:include filename="components/tcp_hollow_cylinder_v1.xacro"/>
-  <xacro:include filename="components/tcp_adaptive_cylinder_v1.xacro"/>
+  <xacro:include filename="components/tcp_shear_v1.xacro"/>
+  <xacro:include filename="components/tcp_bite_shear_v1.xacro"/>
+  <xacro:include filename="components/tcp_adaptive_shear_v1.xacro"/>
   <xacro:include filename="aubo_e5.ros2_control.xacro"/>
   <xacro:arg name="include_table" default="true"/>
@@ -15,7 +16,8 @@
   <xacro:arg name="hardware_mode" default="mock"/>
   <xacro:arg name="robot_ip" default="169.254.10.98"/>
-  <!-- tool_profile: hollow_cylinder_v1 (固定圆柱) | adaptive_cylinder_v1 (自适应圆柱+IMU)。
-       两个独立 if（非 if/else）：未知 profile 名两支都不展开 → 缺 tcp 帧，启动即失败。 -->
-  <xacro:arg name="tool_profile" default="adaptive_cylinder_v1"/>
+  <!-- tool_profile: adaptive_shear_v1 (自适应剪切手+IMU，默认) | bite_shear_v1 (咬合式)
+       | shear_v1 (剪切手)。三个独立 if（非 if/else）：未知 profile 名三支都不展开
+       → 缺 tcp 帧，启动即失败。 -->
+  <xacro:arg name="tool_profile" default="adaptive_shear_v1"/>
   <xacro:property name="tool_profile" value="$(arg tool_profile)"/>
   <xacro:aubo_e5_ros2_control
@@ -33,10 +35,13 @@
   </xacro:if>
   <!-- 末端 TCP 固定关节（URDF 内建，robot_state_publisher 发布，见 components/tcp_<profile>.xacro；
-       帧名冻结，两把工具仅 tool_axis 原点不同） -->
-  <xacro:if value="${tool_profile == 'hollow_cylinder_v1'}">
-    <xacro:aubo_e5_tcp_hollow_cylinder_v1 parent="wrist3_Link"/>
+       帧名冻结，三把剪切手仅 tool_axis 原点/姿态与网格不同） -->
+  <xacro:if value="${tool_profile == 'shear_v1'}">
+    <xacro:aubo_e5_tcp_shear_v1 parent="wrist3_Link"/>
   </xacro:if>
-  <xacro:if value="${tool_profile == 'adaptive_cylinder_v1'}">
-    <xacro:aubo_e5_tcp_adaptive_cylinder_v1 parent="wrist3_Link"/>
+  <xacro:if value="${tool_profile == 'bite_shear_v1'}">
+    <xacro:aubo_e5_tcp_bite_shear_v1 parent="wrist3_Link"/>
+  </xacro:if>
+  <xacro:if value="${tool_profile == 'adaptive_shear_v1'}">
+    <xacro:aubo_e5_tcp_adaptive_shear_v1 parent="wrist3_Link"/>
   </xacro:if>
 </robot>

File: src/aubo_description/urdf/components/tcp.xacro (robot description, xacro)
@@ -3,17 +3,19 @@
   <!-- 末端 TCP 共享底座：帧名冻结（tool_axis/cutting_plane/tcp/sleeve_mouth/tool_body_link），
        SRDF 链 tip、ACM×octomap 豁免名单、技能/重建的三点 TF 验证均按名消费，不得改名。
-       两把工具仅 tool_axis 原点不同，常量由各 wrapper（tcp_<profile>.xacro）持有；
+       2026-09-28 起三把剪切手共用（shear_v1 / bite_shear_v1 / adaptive_shear_v1，替换两把套袋圆柱）：
+       tool_axis 原点/姿态、sleeve_mouth 偏移、网格名由各 wrapper（tcp_<profile>.xacro）传入；
        几何档案：aubo_description/config/<profile>.yaml（改几何改 wrapper 与档案两处）。
-       TCP 姿态：Z = 开口方向，XY = 刀口平面（剪切在该水平面上）。
-       相对法兰 Rx(-90°)，零位开口朝世界 +Z。
-       L_blade=0 → cutting_plane / tcp / sleeve_mouth 同点（顶部）；
-       筒体沿 TCP −Z 长 L_insert=200mm。
+       TCP 姿态：Z = 开口方向，XY = 刀口平面。
+       cutting_plane / tcp 与 tool_axis 同点（刀口深度登记在档案 geometry_m.L_blade）。
+       tool_body_link 直接挂 parent：网格在法兰系（=parent 系）下建模，identity 落位；
+       CAD 原点 = wrist3_Link 原点已数值验证（link6 Ø75 法兰 + STW 快换盘 + 相机族三方叠对）。
+       STEP→网格管线：scripts/step_extract_tool.py + scripts/decimate_export.py。
        不得再用 static_transform_publisher 补发 wrist3_Link→tcp。 -->
-  <xacro:macro name="aubo_e5_tcp" params="parent:=wrist3_Link tcp_xyz:='0 0.0479 0.15107'">
+  <xacro:macro name="aubo_e5_tcp" params="parent:=wrist3_Link tcp_xyz:='0 0 0' tcp_rpy:='-1.5708 0 0' sleeve_mouth_z:=0.0 mesh_stem:=shear_v1 body_rgba:='0.55 0.58 0.62 1.0'">
     <link name="tool_axis"/>
     <joint name="tool_axis_joint" type="fixed">
       <parent link="${parent}"/>
       <child link="tool_axis"/>
-      <origin xyz="${tcp_xyz}" rpy="-1.5708 0 0"/>
+      <origin xyz="${tcp_xyz}" rpy="${tcp_rpy}"/>
     </joint>
     <link name="cutting_plane"/>
@@ -33,42 +35,24 @@
       <parent link="tool_axis"/>
       <child link="sleeve_mouth"/>
-      <origin xyz="0 0 0" rpy="0 0 0"/>
+      <origin xyz="0 0 ${sleeve_mouth_z}" rpy="0 0 0"/>
     </joint>
     <link name="tool_body_link">
-      <!-- 筒在 TCP 下方，沿 −Z；顶部 = TCP -->
+      <!-- 网格在法兰系（parent 系）下建模：identity 挂 parent 即正确落位 -->
       <visual>
-        <origin xyz="0 0 -0.100" rpy="0 0 0"/>
         <geometry>
-          <cylinder radius="0.060" length="0.200"/>
+          <mesh filename="package://aubo_description/meshes/visual/tools/${mesh_stem}.stl"/>
         </geometry>
-        <material name="hollow_cylinder_steel">
-          <color rgba="0.55 0.58 0.62 0.55"/>
-        </material>
-      </visual>
-      <!-- 刀口 / 开口：TCP XY 水平面（圆柱顶部） -->
-      <visual>
-        <origin xyz="0 0 0" rpy="0 0 0"/>
-        <geometry>
-          <cylinder radius="0.060" length="0.003"/>
-        </geometry>
-        <material name="hollow_cylinder_blade">
-          <color rgba="0.75 0.15 0.12 1.0"/>
+        <material name="tool_body_mat">
+          <color rgba="${body_rgba}"/>
         </material>
       </visual>
       <collision>
-        <origin xyz="0 0 -0.100" rpy="0 0 0"/>
         <geometry>
-          <cylinder radius="0.060" length="0.200"/>
-        </geometry>
-      </collision>
-      <collision>
-        <origin xyz="0 0 0" rpy="0 0 0"/>
-        <geometry>
-          <cylinder radius="0.056" length="0.003"/>
+          <mesh filename="package://aubo_description/meshes/collision/tools/${mesh_stem}.stl"/>
         </geometry>
       </collision>
     </link>
     <joint name="tool_body_joint" type="fixed">
-      <parent link="tool_axis"/>
+      <parent link="${parent}"/>
       <child link="tool_body_link"/>
       <origin xyz="0 0 0" rpy="0 0 0"/>

File: src/peach_sim/urdf/harvester_robot.urdf.xacro (robot description, xacro)
@@ -14,8 +14,9 @@
   <xacro:include filename="$(find aubo_description)/urdf/components/camera.xacro"/>
   <xacro:include filename="$(find aubo_description)/urdf/components/quick_changer.xacro"/>
-  <xacro:include filename="$(find aubo_description)/urdf/components/tcp_hollow_cylinder_v1.xacro"/>
-  <xacro:include filename="$(find aubo_description)/urdf/components/tcp_adaptive_cylinder_v1.xacro"/>
+  <xacro:include filename="$(find aubo_description)/urdf/components/tcp_shear_v1.xacro"/>
+  <xacro:include filename="$(find aubo_description)/urdf/components/tcp_bite_shear_v1.xacro"/>
+  <xacro:include filename="$(find aubo_description)/urdf/components/tcp_adaptive_shear_v1.xacro"/>
   <xacro:include filename="tracked_platform.xacro"/>
-  <xacro:arg name="tool_profile" default="adaptive_cylinder_v1"/>
+  <xacro:arg name="tool_profile" default="adaptive_shear_v1"/>
   <xacro:arg name="arm_mount_height" default="0.75"/>
   <xacro:arg name="arm_mount_yaw_deg" default="-32.0"/>
@@ -44,10 +45,13 @@
   <xacro:aubo_e5_camera parent="wrist3_Link"/>
   <xacro:aubo_e5_quick_changer parent="camera_body_link"/>
-  <!-- 两个独立 if（非 if/else）：未知 profile 名两支都不展开 → 缺 tcp 帧，启动即失败 -->
-  <xacro:if value="${tool_profile == 'hollow_cylinder_v1'}">
-    <xacro:aubo_e5_tcp_hollow_cylinder_v1 parent="wrist3_Link"/>
+  <!-- 三个独立 if（非 if/else）：未知 profile 名三支都不展开 → 缺 tcp 帧，启动即失败 -->
+  <xacro:if value="${tool_profile == 'shear_v1'}">
+    <xacro:aubo_e5_tcp_shear_v1 parent="wrist3_Link"/>
   </xacro:if>
-  <xacro:if value="${tool_profile == 'adaptive_cylinder_v1'}">
-    <xacro:aubo_e5_tcp_adaptive_cylinder_v1 parent="wrist3_Link"/>
+  <xacro:if value="${tool_profile == 'bite_shear_v1'}">
+    <xacro:aubo_e5_tcp_bite_shear_v1 parent="wrist3_Link"/>
+  </xacro:if>
+  <xacro:if value="${tool_profile == 'adaptive_shear_v1'}">
+    <xacro:aubo_e5_tcp_adaptive_shear_v1 parent="wrist3_Link"/>
   </xacro:if>
   <!-- 仿真站姿：真机拍照位 photo_joints（field_pregrasp_cases.yaml） -->
