Commit message: test(冻结相机) 战役收口入库
- manipulation 产品修复：staging 种子 IK 分支连续(goal_joints+seeded_ik)、关节目标 Pilz PTP 优先+OMPL 兜底、select_roll 选型期插入 LIN 验证(CONTACT 场景相)、自由规划有界重试；197/197 单测绿，mon11 实测 staging 腕大摆消除(detour 全 1.00)
- 出生即真拍照位(操作员授权 MUST 参数化)：ros2_control.xacro mock_initial_positions 宏参数(缺省=原字面量，无参展开与 HEAD 逐字节等价已证)+urdf.xacro/bringup/peach2_system 透传；操作员裁定真拍照位=global_photo_pose
- photo-move 备用流彻底删除(操作员裁定该流是错的)：drive/run 脚本、photo_pose.py、SRDF frozen_photo_pose 位
- rviz2 可视化修复：offscreen 强设移除+moveit.launch.py rviz 开关；GLX 100 次/轮崩溃根除
- 真拍照位数据边界定论：本 bag(静止场景)FULL 插入出可达球三轮确定性复现；PREGRASP 通过档 cycle~21s
- 测试报告 §5.8-5.14/截图存证/账本文本层入库；testing.md/testing-log/README 同轮对齐

File: src/aubo_description/urdf/aubo_e5.ros2_control.xacro (robot description, xacro)
@@ -32,5 +32,11 @@
     dedup_threshold:=0.000001
     state_timeout_ms:=200
-    auto_power_on:=false">
+    auto_power_on:=false
+    mock_initial_positions:='0.425083,0.195177,1.677740,1.461739,-0.500161,0.038621'">
+    <!-- 2026-10-09 操作员授权的默认不变参数化：mock 六关节初值按
+         shoulder,upperArm,foreArm,wrist1,wrist2,wrist3 顺序取逗号串元素；
+         缺省串与原字面量逐位相同（展开结果不变）。仅 mock 分支使用，
+         real 分支不读初值。 -->
+    <xacro:property name="mock_q" value="${mock_initial_positions.split(',')}"/>
     <ros2_control name="${name}" type="system">
       <hardware>
@@ -68,5 +74,5 @@
         <command_interface name="position"/>
         <state_interface name="position">
-          <param name="initial_value">0.425083</param>
+          <param name="initial_value">${mock_q[0]}</param>
         </state_interface>
         <state_interface name="velocity"/>
@@ -75,5 +81,5 @@
         <command_interface name="position"/>
         <state_interface name="position">
-          <param name="initial_value">0.195177</param>
+          <param name="initial_value">${mock_q[1]}</param>
         </state_interface>
         <state_interface name="velocity"/>
@@ -82,5 +88,5 @@
         <command_interface name="position"/>
         <state_interface name="position">
-          <param name="initial_value">1.677740</param>
+          <param name="initial_value">${mock_q[2]}</param>
         </state_interface>
         <state_interface name="velocity"/>
@@ -89,5 +95,5 @@
         <command_interface name="position"/>
         <state_interface name="position">
-          <param name="initial_value">1.461739</param>
+          <param name="initial_value">${mock_q[3]}</param>
         </state_interface>
         <state_interface name="velocity"/>
@@ -96,5 +102,5 @@
         <command_interface name="position"/>
         <state_interface name="position">
-          <param name="initial_value">-0.500161</param>
+          <param name="initial_value">${mock_q[4]}</param>
         </state_interface>
         <state_interface name="velocity"/>
@@ -103,5 +109,5 @@
         <command_interface name="position"/>
         <state_interface name="position">
-          <param name="initial_value">0.038621</param>
+          <param name="initial_value">${mock_q[5]}</param>
         </state_interface>
         <state_interface name="velocity"/>

File: src/aubo_description/urdf/aubo_e5.urdf.xacro (robot description, xacro)
@@ -21,8 +21,12 @@
   <xacro:arg name="tool_profile" default="adaptive_shear_v1"/>
   <xacro:property name="tool_profile" value="$(arg tool_profile)"/>
+  <!-- 2026-10-09 操作员授权：mock 六关节初值（shoulder..wrist3 逗号串），缺省=原字面量 -->
+  <xacro:arg name="mock_initial_positions"
+             default="0.425083,0.195177,1.677740,1.461739,-0.500161,0.038621"/>
   <xacro:aubo_e5_ros2_control
     name="AuboE5System"
     hardware_mode="$(arg hardware_mode)"
-    robot_ip="$(arg robot_ip)"/>
+    robot_ip="$(arg robot_ip)"
+    mock_initial_positions="$(arg mock_initial_positions)"/>
   <xacro:if value="$(arg include_table)">
     <xacro:aubo_e5_table parent="world"/>
