Commit message: feat(2026-10-08) 冻结相机抓取验证、时效/命令门修正、orchard_nav 与 v1/v2 架构图入库
同轮收口：peach2/peach 冻结回放抓取系统测；target_model/core/gate 正确性与 v1 退出线程；peach_sim 履带 Nav2 巡园；方案与架构图；runs 文本账本随仓（bag 二进制仍本地）。

Co-authored-by: Cursor <cursoragent@cursor.com>

File: src/peach_sim/urdf/harvester_robot.urdf.xacro (robot description, xacro)
@@ -2,20 +2,17 @@
 <robot name="peach_harvester" xmlns:xacro="http://www.ros.org/wiki/xacro">
   <!-- 采摘工位整机：开源履带底盘改型 + AUBO E5 + 腕载相机 + 快换 + 套袋刀。
-    帧契约：`world` 与 `base_link` 由 aubo_description/urdf/aubo_e5.urdf 恒等连接
-    （= 臂座，与真机栈 /tf_static world→base 同构）；履带车挂在 `world` 下方
-    arm_mount_height、反向转台偏航。gz 侧模型原点 = `world` = 臂座。
-    仿真站姿：六关节由 gz JointPositionController 钉在真机拍照位
-    （photo_joints，来源 src/peach_arm/test/fixtures/field_pregrasp_cases.yaml），
-    关节状态经 gz JointStatePublisher → ros_gz_bridge 进 /joint_states，
-    robot_state_publisher 出的 TF 与 gz 内几何一致。
-    不改 aubo_description 只读面（aubo_e5.ros2_control.xacro / bringup.launch.py）：
-    gz_ros2_control 接管关节属后续轮。 -->
-  <xacro:include filename="$(find aubo_description)/urdf/aubo_e5.urdf"/>
-  <xacro:include filename="$(find aubo_description)/urdf/components/camera.xacro"/>
-  <xacro:include filename="$(find aubo_description)/urdf/components/quick_changer.xacro"/>
-  <xacro:include filename="$(find aubo_description)/urdf/components/tcp_shear_v1.xacro"/>
-  <xacro:include filename="$(find aubo_description)/urdf/components/tcp_bite_shear_v1.xacro"/>
-  <xacro:include filename="$(find aubo_description)/urdf/components/tcp_adaptive_shear_v1.xacro"/>
-  <xacro:include filename="tracked_platform.xacro"/>
+    两模式共享 config/orchard.yaml 的 platform.* 尺寸注入（launch 按 yaml 传参）：
+    mobile:=false（默认，锚定建模轮）：含完整臂链。帧契约与真机栈同构——
+    `world` 与 `base_link` 由 aubo_e5.urdf 恒等连接；URDF→SDF 后 world_joint
+    把整机焊在仿真世界（固定座语义，整车不可驾驶）；履带车挂 `world` 下方
+    arm_mount_height、反向转台偏航。六关节由 gz JointPositionController 钉在
+    真机拍照位（photo_joints，field_pregrasp_cases.yaml）。
+    mobile:=true（自主导航轮，REP-105）：不含臂链（world_joint 的世界锚定
+    无法在只读 aubo_description 之外解除；本轮导航不动臂）。根 =
+    platform_base_link，spawn 落地 z=0；驱动 = gz DiffDrive（履带滚筒轮），
+    发布 /odom 与 odom→platform_base_link TF；帧树
+    map→odom→platform_base_link→{left,right}_track/lidar_mount，
+    map→odom 由 Nav2 AMCL/SLAM 发布。
+    不改 aubo_description 只读面；gz_ros2_control 接臂属后续轮。 -->
   <xacro:arg name="tool_profile" default="adaptive_shear_v1"/>
   <xacro:arg name="arm_mount_height" default="0.75"/>
@@ -30,5 +27,16 @@
   <xacro:arg name="track_separation" default="0.56"/>
   <xacro:arg name="hold_arm" default="true"/>
+  <xacro:arg name="mobile" default="false"/>
   <xacro:property name="tool_profile" value="$(arg tool_profile)"/>
+  <xacro:property name="mobile" value="$(arg mobile)"/>
+  <xacro:include filename="tracked_platform.xacro"/>
+  <xacro:unless value="${mobile}">
+    <xacro:include filename="$(find aubo_description)/urdf/aubo_e5.urdf"/>
+    <xacro:include filename="$(find aubo_description)/urdf/components/camera.xacro"/>
+    <xacro:include filename="$(find aubo_description)/urdf/components/quick_changer.xacro"/>
+    <xacro:include filename="$(find aubo_description)/urdf/components/tcp_shear_v1.xacro"/>
+    <xacro:include filename="$(find aubo_description)/urdf/components/tcp_bite_shear_v1.xacro"/>
+    <xacro:include filename="$(find aubo_description)/urdf/components/tcp_adaptive_shear_v1.xacro"/>
+  </xacro:unless>
   <xacro:peach_tracked_platform
     parent="world"
@@ -42,38 +50,42 @@
     track_width="$(arg track_width)"
     track_height="$(arg track_height)"
-    track_separation="$(arg track_separation)"/>
-  <xacro:aubo_e5_camera parent="wrist3_Link"/>
-  <xacro:aubo_e5_quick_changer parent="camera_body_link"/>
-  <!-- 三个独立 if（非 if/else）：未知 profile 名三支都不展开 → 缺 tcp 帧，启动即失败 -->
-  <xacro:if value="${tool_profile == 'shear_v1'}">
-    <xacro:aubo_e5_tcp_shear_v1 parent="wrist3_Link"/>
-  </xacro:if>
-  <xacro:if value="${tool_profile == 'bite_shear_v1'}">
-    <xacro:aubo_e5_tcp_bite_shear_v1 parent="wrist3_Link"/>
-  </xacro:if>
-  <xacro:if value="${tool_profile == 'adaptive_shear_v1'}">
-    <xacro:aubo_e5_tcp_adaptive_shear_v1 parent="wrist3_Link"/>
-  </xacro:if>
-  <!-- 仿真站姿：真机拍照位 photo_joints（field_pregrasp_cases.yaml） -->
-  <xacro:macro name="hold_joint" params="name value">
-    <gazebo>
-      <plugin name="gz::sim::systems::JointPositionController"
-              filename="gz-sim-joint-position-controller-system">
-        <joint_name>${name}</joint_name>
-        <initial_position>${value}</initial_position>
-        <use_velocity_commands>1</use_velocity_commands>
-        <cmd_max>1.5</cmd_max>
-      </plugin>
-    </gazebo>
-  </xacro:macro>
-  <xacro:if value="$(arg hold_arm)">
-    <xacro:hold_joint name="shoulder_joint" value="0.425083"/>
-    <xacro:hold_joint name="upperArm_joint" value="0.195177"/>
-    <xacro:hold_joint name="foreArm_joint" value="1.677740"/>
-    <xacro:hold_joint name="wrist1_joint" value="1.461739"/>
-    <xacro:hold_joint name="wrist2_joint" value="-0.500161"/>
-    <xacro:hold_joint name="wrist3_joint" value="0.038621"/>
-  </xacro:if>
-  <!-- 关节状态出 gz（ros_gz_bridge: gz.msgs.Model → sensor_msgs/JointState） -->
+    track_separation="$(arg track_separation)"
+    mobile="$(arg mobile)"/>
+  <xacro:unless value="${mobile}">
+    <xacro:aubo_e5_camera parent="wrist3_Link"/>
+    <xacro:aubo_e5_quick_changer parent="camera_body_link"/>
+    <!-- 三个独立 if（非 if/else）：未知 profile 名三支都不展开 → 缺 tcp 帧，启动即失败 -->
+    <xacro:if value="${tool_profile == 'shear_v1'}">
+      <xacro:aubo_e5_tcp_shear_v1 parent="wrist3_Link"/>
+    </xacro:if>
+    <xacro:if value="${tool_profile == 'bite_shear_v1'}">
+      <xacro:aubo_e5_tcp_bite_shear_v1 parent="wrist3_Link"/>
+    </xacro:if>
+    <xacro:if value="${tool_profile == 'adaptive_shear_v1'}">
+      <xacro:aubo_e5_tcp_adaptive_shear_v1 parent="wrist3_Link"/>
+    </xacro:if>
+    <!-- 仿真站姿：真机拍照位 photo_joints（field_pregrasp_cases.yaml） -->
+    <xacro:macro name="hold_joint" params="name value">
+      <gazebo>
+        <plugin name="gz::sim::systems::JointPositionController"
+                filename="gz-sim-joint-position-controller-system">
+          <joint_name>${name}</joint_name>
+          <initial_position>${value}</initial_position>
+          <use_velocity_commands>1</use_velocity_commands>
+          <cmd_max>1.5</cmd_max>
+        </plugin>
+      </gazebo>
+    </xacro:macro>
+    <xacro:if value="$(arg hold_arm)">
+      <xacro:hold_joint name="shoulder_joint" value="0.425083"/>
+      <xacro:hold_joint name="upperArm_joint" value="0.195177"/>
+      <xacro:hold_joint name="foreArm_joint" value="1.677740"/>
+      <xacro:hold_joint name="wrist1_joint" value="1.461739"/>
+      <xacro:hold_joint name="wrist2_joint" value="-0.500161"/>
+      <xacro:hold_joint name="wrist3_joint" value="0.038621"/>
+    </xacro:if>
+  </xacro:unless>
+  <!-- 关节状态出 gz（ros_gz_bridge: gz.msgs.Model → sensor_msgs/JointState）；
+       mobile 模式发布履带滚筒关节角，锚定模式发布臂关节角 -->
   <gazebo>
     <plugin name="gz::sim::systems::JointStatePublisher"

File: src/peach_sim/urdf/tracked_platform.xacro (robot description, xacro)
@@ -6,12 +6,19 @@
     两端圆柱，ODE 摩擦 mu 0.7 / mu2 150 / fdir1 0 1 0（横向高摩擦近似履带）。
     默认尺寸即 config/orchard.yaml 的 platform.*（launch 按 yaml 注入，测试对账）。
-    帧约定：platform_base_link 在两履带中线、接地平面（z=0），+X 沿行行驶方向；
-    车体挂在臂座（parent，= base_link）下方 arm_mount_height、反向转台偏航。
-    本轮是场景建模：整车经 world_joint 锚在作业位（见 harvester_robot.urdf.xacro），
-    履带驱动（gz::sim::systems::TrackedVehicle + TrackController，见官方示例
-    ~L1060）与线控留待移动化那轮，届时一并把 world 锚点换成 map→odom→base_link。
+    帧约定：platform_base_link 在两履带中线、接地平面（z=0），+X 沿行行驶方向。
+    mobile:=true 时 platform_base_link 即 URDF/gz 模型根（臂链不含入——
+    aubo world_joint 会把整机焊死在世界系，见 harvester_robot.urdf.xacro）；
+    mobile:=false 时车体挂在臂座（parent，= base_link）下方 arm_mount_height、
+    反向转台偏航，world 为模型根（SDF 保留帧名，非根会被 gz 拒建）。
+    mobile:=false（默认，锚定建模轮）：整车锚在作业位，履带不可驾驶。
+    mobile:=true（自主导航轮，REP-105）：履带 = 滚筒驱动轮（continuous 关节 +
+    圆柱碰撞体，盒体仅视觉），gz DiffDrive 驱动（官方 TB3/TB4 仿真同款），
+    发布 /odom 与 odom→platform_base_link TF（关节积分里程计）；
+    mobile 时转台偏航由 launch 归零，world 与 platform 同向无恒定偏差。
+    前桅杆 2D 激光（±95°，车体自遮挡裁剪后）供 Nav2 使用；
+    map→odom 由 AMCL/SLAM 发布，不在此 URDF。
     数值入参一律字符串进、float() 出（xacro 属性默认是字符串，直接相加会拼接）。 -->
   <xacro:macro name="peach_tracked_platform"
-               params="parent arm_mount_height arm_mount_yaw_deg body_x body_y body_z body_bottom track_length track_width track_height track_separation">
+               params="parent arm_mount_height arm_mount_yaw_deg body_x body_y body_z body_bottom track_length track_width track_height track_separation mobile:=false">
     <xacro:property name="mount_h" value="${float(arm_mount_height)}"/>
     <xacro:property name="mount_yaw" value="${-float(arm_mount_yaw_deg) * pi / 180.0}"/>
@@ -67,9 +74,13 @@
       </collision>
     </link>
-    <joint name="platform_mount" type="fixed">
-      <parent link="${parent}"/>
-      <child link="platform_base_link"/>
-      <origin xyz="0 0 ${-mount_h}" rpy="0 0 ${mount_yaw}"/>
-    </joint>
+    <!-- 层级：锚定 = world（臂座，模型根）→ platform_base_link → 履带/桅杆；
+       mobile = platform_base_link 即根（无臂链、无 world 链接） -->
+    <xacro:unless value="${mobile}">
+      <joint name="platform_mount" type="fixed">
+        <parent link="${parent}"/>
+        <child link="platform_base_link"/>
+        <origin xyz="0 0 ${-mount_h}" rpy="0 0 ${mount_yaw}"/>
+      </joint>
+    </xacro:unless>
     <xacro:macro name="track_unit" params="name side">
       <link name="${name}">
@@ -88,10 +99,22 @@
           </material>
         </visual>
-        <collision name="${name}_collision">
-          <origin xyz="0 0 0" rpy="${pi / 2.0} 0 ${pi / 2.0}"/>
-          <geometry>
-            <box size="${tw} ${th} ${tl}"/>
-          </geometry>
-        </collision>
+        <xacro:if value="${mobile}">
+          <!-- mobile：滚筒碰撞体（轴 Y、半径 th/2、长 tl）——DiffDrive 关节驱动下
+               平滑滚动，等效履带接地印迹；盒体仅作视觉 -->
+          <collision name="${name}_collision">
+            <origin xyz="0 0 0" rpy="${pi / 2.0} 0 0"/>
+            <geometry>
+              <cylinder radius="${wheel_r}" length="${tl}"/>
+            </geometry>
+          </collision>
+        </xacro:if>
+        <xacro:unless value="${mobile}">
+          <collision name="${name}_collision">
+            <origin xyz="0 0 0" rpy="${pi / 2.0} 0 ${pi / 2.0}"/>
+            <geometry>
+              <box size="${tw} ${th} ${tl}"/>
+            </geometry>
+          </collision>
+        </xacro:unless>
         <visual name="${name}_wheel_front">
           <origin xyz="${wheel_x} 0 0" rpy="${pi / 2.0} 0 0"/>
@@ -121,18 +144,142 @@
         </collision>
       </link>
-      <joint name="${name}_mount" type="fixed">
-        <parent link="platform_base_link"/>
-        <child link="${name}"/>
-        <origin xyz="0 ${side * ts / 2.0} ${th / 2.0}" rpy="0 0 0"/>
-      </joint>
-      <!-- 履带摩擦（官方示例口径）：横向高摩擦、纵向低摩擦近似履带推进 -->
-      <gazebo reference="${name}">
-        <mu1>0.7</mu1>
-        <mu2>150</mu2>
-        <fdir1>0 1 0</fdir1>
-      </gazebo>
+      <!-- 履带挂接：mobile 用 continuous 转动关节当驱动轮——URDF→SDF 会把固定
+           关节子链接合并进父链接（fixed-joint lumping），履带不成其为独立链接、
+           无从驱动（冒烟实测固定关节时 TrackController 表面速度不出牵引）。
+           锚定模式仍用固定关节。 -->
+      <xacro:if value="${mobile}">
+        <joint name="${name}_mount" type="continuous">
+          <parent link="platform_base_link"/>
+          <child link="${name}"/>
+          <origin xyz="0 ${side * ts / 2.0} ${th / 2.0}" rpy="0 0 0"/>
+          <axis xyz="0 1 0"/>
+          <dynamics damping="0.05" friction="0.0"/>
+          <limit effort="1e5" velocity="20"/>
+        </joint>
+      </xacro:if>
+      <xacro:unless value="${mobile}">
+        <joint name="${name}_mount" type="fixed">
+          <parent link="platform_base_link"/>
+          <child link="${name}"/>
+          <origin xyz="0 ${side * ts / 2.0} ${th / 2.0}" rpy="0 0 0"/>
+        </joint>
+      </xacro:unless>
+      <!-- 履带摩擦：gz-physics dartsim 对未显式声明的碰撞不保证默认摩擦
+           （官方 TB3/TB4 轮子全部显式 <surface><friction>）。
+           mobile：各向同性 mu 1/1（TB3 轮口径，无 fdir1——圆柱碰撞系里
+           fdir1 会指向竖直方向、破坏滚动牵引，冒烟实测）。
+           锚定：官方履带口径（fdir1 车体横向 mu 0.7 / 纵向 mu2 150）。 -->
+      <xacro:if value="${mobile}">
+        <gazebo reference="${name}">
+          <mu1>1.0</mu1>
+          <mu2>1.0</mu2>
+        </gazebo>
+      </xacro:if>
+      <xacro:unless value="${mobile}">
+        <gazebo reference="${name}">
+          <mu1>0.7</mu1>
+          <mu2>150</mu2>
+          <fdir1>0 1 0</fdir1>
+        </gazebo>
+      </xacro:unless>
     </xacro:macro>
     <xacro:track_unit name="left_track" side="1.0"/>
     <xacro:track_unit name="right_track" side="-1.0"/>
+    <xacro:if value="${mobile}">
+      <!-- 前桅杆 2D 激光：z=0.45 穿树干区（干高 0.50–0.65 与棚架立柱均可见），
+           FOV ±95°——车体（z 0.22–0.54，前缘 x=0.525）对后向扇区自遮挡，
+           超出 ±101° 的射线会打到自身车体，这里直接不发射。 -->
+      <xacro:property name="lidar_x" value="${0.5 * bx + 0.055}"/>
+      <xacro:property name="lidar_z" value="${0.45}"/>
+      <link name="lidar_mount">
+        <inertial>
+          <origin xyz="0 0 0" rpy="0 0 0"/>
+          <mass value="0.3"/>
+          <inertia ixx="0.0004" ixy="0.0" ixz="0.0" iyy="0.0004" iyz="0.0" izz="0.0006"/>
+        </inertial>
+        <visual name="lidar_head_visual">
+          <origin xyz="0 0 0" rpy="0 0 0"/>
+          <geometry>
+            <cylinder radius="0.025" length="0.035"/>
+          </geometry>
+          <material name="lidar_dark">
+            <color rgba="0.12 0.12 0.12 1.0"/>
+          </material>
+        </visual>
+        <collision name="lidar_head_collision">
+          <origin xyz="0 0 0" rpy="0 0 0"/>
+          <geometry>
+            <cylinder radius="0.025" length="0.035"/>
+          </geometry>
+        </collision>
+        <visual name="lidar_pole_visual">
+          <!-- 触地桅杆仅视觉（低模）：不给碰撞，避免前端附加摩擦点干扰履带驱动 -->
+          <origin xyz="0 0 ${-lidar_z / 2.0}" rpy="0 0 0"/>
+          <geometry>
+            <cylinder radius="0.012" length="${lidar_z}"/>
+          </geometry>
+          <material name="lidar_dark"/>
+        </visual>
+      </link>
+      <joint name="lidar_mount_joint" type="fixed">
+        <parent link="platform_base_link"/>
+        <child link="lidar_mount"/>
+        <origin xyz="${lidar_x} 0 ${lidar_z}" rpy="0 0 0"/>
+      </joint>
+      <gazebo reference="lidar_mount">
+        <sensor name="orchard_scan" type="gpu_lidar">
+          <pose>0 0 0 0 0 0</pose>
+          <topic>/scan</topic>
+          <gz_frame_id>lidar_mount</gz_frame_id>
+          <update_rate>10</update_rate>
+          <always_on>1</always_on>
+          <visualize>true</visualize>
+          <lidar>
+            <scan>
+              <horizontal>
+                <samples>190</samples>
+                <resolution>1</resolution>
+                <min_angle>${-95.0 * pi / 180.0}</min_angle>
+                <max_angle>${95.0 * pi / 180.0}</max_angle>
+              </horizontal>
+            </scan>
+            <range>
+              <min>0.25</min>
+              <max>12.0</max>
+              <resolution>0.01</resolution>
+            </range>
+            <noise>
+              <type>gaussian</type>
+              <mean>0.0</mean>
+              <stddev>0.01</stddev>
+            </noise>
+          </lidar>
+        </sensor>
+      </gazebo>
+      <!-- 底盘驱动：gz DiffDrive（官方 TB3/TB4 仿真同款，gz-sim 8 URDF 路径
+           验证可用）。左右履带 = 滚筒驱动轮（continuous 关节），odom 由关节
+           角积分。履带表面速度方案（TrackedVehicle+TrackController）在 8.15
+           URDF→SDF 路径上冒烟实测不出牵引（指令链通、整车不动），留待原生
+           SDF 模型轮再试。mobile 时转台偏航归零 → world 与 platform_base_link
+           同向，child_frame_id 取 platform_base_link 无恒定偏差。 -->
+      <gazebo>
+        <plugin name="gz::sim::systems::DiffDrive"
+                filename="gz-sim-diff-drive-system">
+          <left_joint>left_track_mount</left_joint>
+          <right_joint>right_track_mount</right_joint>
+          <wheel_separation>${ts}</wheel_separation>
+          <wheel_radius>${wheel_r}</wheel_radius>
+          <topic>/cmd_vel</topic>
+          <odom_topic>/odom</odom_topic>
+          <odom_publish_frequency>50</odom_publish_frequency>
+          <tf_topic>/tf</tf_topic>
+          <frame_id>odom</frame_id>
+          <child_frame_id>platform_base_link</child_frame_id>
+          <max_linear_acceleration>1.0</max_linear_acceleration>
+          <max_linear_deceleration>1.0</max_linear_deceleration>
+          <max_angular_acceleration>2.0</max_angular_acceleration>
+        </plugin>
+      </gazebo>
+    </xacro:if>
   </xacro:macro>
 </robot>
