Commit message: chore: 工作区打包脚本 + peach_sim 固定工位 BUNKER 外观 + ivg foxglove 零字段服务修复入库
- scripts/pack_workspace.sh：工作区迁移打包脚本（源码+资产+git 历史；排除
  编译产物/venv/会话输出/可重下大件；reconstruction/output/ 只随包带 git
  跟踪验证产物；打包白名单含 scripts/ 与 web 前端 vendor 发行件），根
  README 同轮补「打包迁移」一节
- peach_sim：固定工位改用 BUNKER Pro 2 彩色底盘外观（来源 AgileX
  ugv_gazebo_sim @27633a9 BSD；bunker_chassis.glb + 源 STL + SHA256 +
  重导出命令见 meshes/BUNKER_SOURCE.md；blender/color_bunker.py 着色脚本）；
  默认 tool_profile 改 bite_shear_v1（launch 与 xacro 同轮）；field_no_grass
  平行光 intensity 4→1；tracked_platform.xacro 固定工位用 BUNKER 网格、
  导航模式保留低模；README 与包级 architecture.md 同轮收口（新增 Gazebo
  模型不可见定位节）
- ivg_foxglove_bridge：generic_client 零字段 srv 请求修复——请求 CDR
  payload ≤4B（仅封装头）时跳过 rmw_deserialize、直接发送 default-init
  实例，规避 rosidl 空结构占位成员反序列化越界抛 Fast CDR 异常
  （ListControllers/GetCurrentState/RunLatteWorkflow 等零字段服务恢复可用）；
  VENDOR_PROVENANCE.md 同轮记录

注：重渲染版 field_no_grass.glb（650152048 字节、压缩后 373.6MB）超 Gitee
单文件 100MB 配额被拒，本次不入库，保留为本地未提交改动；仓库内仍为
149909776 字节旧版。

File: src/peach_sim/urdf/harvester_robot.urdf.xacro (robot description, xacro)
@@ -15,5 +15,5 @@
     map→odom 由 Nav2 AMCL/SLAM 发布。
     不改 aubo_description 只读面；gz_ros2_control 接臂属后续轮。 -->
-  <xacro:arg name="tool_profile" default="adaptive_shear_v1"/>
+  <xacro:arg name="tool_profile" default="bite_shear_v1"/>
   <xacro:arg name="arm_mount_height" default="0.75"/>
   <xacro:arg name="arm_mount_yaw_deg" default="-32.0"/>
@@ -55,5 +55,5 @@
     <xacro:aubo_e5_camera parent="wrist3_Link"/>
     <xacro:aubo_e5_quick_changer parent="camera_body_link"/>
-    <!-- 三个独立 if（非 if/else）：未知 profile 名三支都不展开 → 缺 tcp 帧，启动即失败 -->
+    <!-- 三种 peach 真实末端各自展开，默认球形环抱的 bite_shear_v1。 -->
     <xacro:if value="${tool_profile == 'shear_v1'}">
       <xacro:aubo_e5_tcp_shear_v1 parent="wrist3_Link"/>

File: src/peach_sim/urdf/tracked_platform.xacro (robot description, xacro)
@@ -1,5 +1,5 @@
 <?xml version="1.0"?>
 <robot xmlns:xacro="http://www.ros.org/wiki/xacro">
-  <!-- 果园采摘工位履带底盘（低模）。
+  <!-- 果园采摘工位履带底盘（固定工位为 BUNKER Pro 2 彩色网格；导航为低模）。
     几何与履带摩擦参数改自 Gazebo Sim 官方示例 worlds/tracked_vehicle_simple.sdf
     的 simple_tracked 模型（gazebosim/gz-sim，Apache-2.0）：双履带 = 箱体 +
@@ -42,13 +42,24 @@
         <inertia ixx="4.05" ixy="0.0" ixz="0.0" iyy="12.05" iyz="0.0" izz="14.05"/>
       </inertial>
-      <visual name="body_visual">
-        <origin xyz="0 0 ${body_cz}" rpy="0 0 0"/>
-        <geometry>
-          <box size="${bx} ${by} ${bz}"/>
-        </geometry>
-        <material name="platform_gray">
-          <color rgba="0.55 0.57 0.55 1.0"/>
-        </material>
-      </visual>
+      <xacro:unless value="${mobile}">
+        <!-- BUNKER 外观网格：带颜色的车体/履带；碰撞仍用下面的简单代理。 -->
+        <visual name="bunker_chassis_visual">
+          <geometry>
+            <mesh filename="package://peach_sim/meshes/bunker_chassis.glb"
+                  scale="${bx / 1.05} ${(ts + tw) / 0.71} ${(bb + bz) / 0.54}"/>
+          </geometry>
+        </visual>
+      </xacro:unless>
+      <xacro:if value="${mobile}">
+        <visual name="body_visual">
+          <origin xyz="0 0 ${body_cz}" rpy="0 0 0"/>
+          <geometry>
+            <box size="${bx} ${by} ${bz}"/>
+          </geometry>
+          <material name="platform_gray">
+            <color rgba="0.55 0.57 0.55 1.0"/>
+          </material>
+        </visual>
+      </xacro:if>
       <collision name="body_collision">
         <origin xyz="0 0 ${body_cz}" rpy="0 0 0"/>
@@ -90,13 +101,15 @@
           <inertia ixx="0.30" ixy="0.0" ixz="0.0" iyy="1.60" iyz="0.0" izz="1.45"/>
         </inertial>
-        <visual name="${name}_visual">
-          <origin xyz="0 0 0" rpy="${pi / 2.0} 0 ${pi / 2.0}"/>
-          <geometry>
-            <box size="${tw} ${th} ${tl}"/>
-          </geometry>
-          <material name="${name}_black">
-            <color rgba="0.16 0.16 0.16 1.0"/>
-          </material>
-        </visual>
+        <xacro:if value="${mobile}">
+          <visual name="${name}_visual">
+            <origin xyz="0 0 0" rpy="${pi / 2.0} 0 ${pi / 2.0}"/>
+            <geometry>
+              <box size="${tw} ${th} ${tl}"/>
+            </geometry>
+            <material name="${name}_black">
+              <color rgba="0.16 0.16 0.16 1.0"/>
+            </material>
+          </visual>
+        </xacro:if>
         <xacro:if value="${mobile}">
           <!-- mobile：滚筒碰撞体（轴 Y、半径 th/2、长 tl）——DiffDrive 关节驱动下
@@ -117,11 +130,13 @@
           </collision>
         </xacro:unless>
-        <visual name="${name}_wheel_front">
-          <origin xyz="${wheel_x} 0 0" rpy="${pi / 2.0} 0 0"/>
-          <geometry>
-            <cylinder radius="${wheel_r}" length="${tw}"/>
-          </geometry>
-          <material name="${name}_black"/>
-        </visual>
+        <xacro:if value="${mobile}">
+          <visual name="${name}_wheel_front">
+            <origin xyz="${wheel_x} 0 0" rpy="${pi / 2.0} 0 0"/>
+            <geometry>
+              <cylinder radius="${wheel_r}" length="${tw}"/>
+            </geometry>
+            <material name="${name}_black"/>
+          </visual>
+        </xacro:if>
         <collision name="${name}_wheel_front_collision">
           <origin xyz="${wheel_x} 0 0" rpy="${pi / 2.0} 0 0"/>
@@ -130,11 +145,13 @@
           </geometry>
         </collision>
-        <visual name="${name}_wheel_rear">
-          <origin xyz="${-wheel_x} 0 0" rpy="${pi / 2.0} 0 0"/>
-          <geometry>
-            <cylinder radius="${wheel_r}" length="${tw}"/>
-          </geometry>
-          <material name="${name}_black"/>
-        </visual>
+        <xacro:if value="${mobile}">
+          <visual name="${name}_wheel_rear">
+            <origin xyz="${-wheel_x} 0 0" rpy="${pi / 2.0} 0 0"/>
+            <geometry>
+              <cylinder radius="${wheel_r}" length="${tw}"/>
+            </geometry>
+            <material name="${name}_black"/>
+          </visual>
+        </xacro:if>
         <collision name="${name}_wheel_rear_collision">
           <origin xyz="${-wheel_x} 0 0" rpy="${pi / 2.0} 0 0"/>

Commit message: fix(peach_sim): 无草整园 GLB 重导出修复 90° 立墙 + 臂直接落底盘无垫台
- field_no_grass.glb 用 v10 脚本(export_yup=False)重导出为 Z-up 顶点(621M,
  --decimate 0.25)：旧 143M 是 fe79b3a 期 yup=True 导出的 Y-up 数据，在本机
  Z-up 直读链上立成 90° 墙(v10 修复了脚本但工件未随之重导出)
- 臂座高度 0.75→0.54=车体顶面(body_bottom+body_z)，去掉 0.21m 垫台方块；
  tracked_platform xacro 垫台高度≤0 不再生成；params 校验放宽为低于车体
  顶面才报错(=顶面即无垫台直落)
- scene.py 袋底现场窗钳制从写死[1.27,1.45]改为随臂座平移(+0.52~0.71)；
  bag.bottom_height [1.30,1.42]→[1.09,1.21] 同步下移保现场相对包络
- generate_orchard 重生成 world/manifest；maps 确定性不变
- XML 解析加固：xmlsafe.parse_xml 拒 DTD/ENTITY，替换 preview/test_scene
  裸 ET.fromstring（Mimosa 高危拦截项）
- doc/architecture.md 臂座口径同轮更新；scene+params 测试 25/25 绿

File: src/peach_sim/urdf/harvester_robot.urdf.xacro (robot description, xacro)
@@ -16,5 +16,5 @@
     不改 aubo_description 只读面；gz_ros2_control 接臂属后续轮。 -->
   <xacro:arg name="tool_profile" default="bite_shear_v1"/>
-  <xacro:arg name="arm_mount_height" default="0.75"/>
+  <xacro:arg name="arm_mount_height" default="0.54"/>
   <xacro:arg name="arm_mount_yaw_deg" default="-32.0"/>
   <xacro:arg name="body_x" default="1.05"/>

File: src/peach_sim/urdf/tracked_platform.xacro (robot description, xacro)
@@ -34,4 +34,5 @@
     <xacro:property name="body_cz" value="${bb + bz / 2.0}"/>
     <xacro:property name="mount_cz" value="${(deck_top + mount_h) / 2.0}"/>
+    <xacro:property name="mount_t" value="${mount_h - deck_top}"/>
     <xacro:property name="wheel_x" value="${tl / 2.0 - th / 2.0}"/>
     <xacro:property name="wheel_r" value="${th / 2.0}"/>
@@ -68,20 +69,23 @@
         </geometry>
       </collision>
-      <!-- 臂安装座（车体顶面 → base_link 离地高度） -->
-      <visual name="mount_visual">
-        <origin xyz="0 0 ${mount_cz}" rpy="0 0 0"/>
-        <geometry>
-          <box size="0.20 0.20 ${mount_h - deck_top}"/>
-        </geometry>
-        <material name="mount_gray">
-          <color rgba="0.45 0.45 0.48 1.0"/>
-        </material>
-      </visual>
-      <collision name="mount_collision">
-        <origin xyz="0 0 ${mount_cz}" rpy="0 0 0"/>
-        <geometry>
-          <box size="0.20 0.20 ${mount_h - deck_top}"/>
-        </geometry>
-      </collision>
+      <!-- 臂安装座（车体顶面 → base_link 离地高度）；mount_t≤0 时臂直接落
+           车体顶面，不生成垫台（零高盒退化，gz 不收） -->
+      <xacro:if value="${mount_t > 1e-9}">
+        <visual name="mount_visual">
+          <origin xyz="0 0 ${mount_cz}" rpy="0 0 0"/>
+          <geometry>
+            <box size="0.20 0.20 ${mount_t}"/>
+          </geometry>
+          <material name="mount_gray">
+            <color rgba="0.45 0.45 0.48 1.0"/>
+          </material>
+        </visual>
+        <collision name="mount_collision">
+          <origin xyz="0 0 ${mount_cz}" rpy="0 0 0"/>
+          <geometry>
+            <box size="0.20 0.20 ${mount_t}"/>
+          </geometry>
+        </collision>
+      </xacro:if>
     </link>
     <!-- 层级：锚定 = world（臂座，模型根）→ platform_base_link → 履带/桅杆；
