Commit message: chore: 2026-10-12 全同步收口——peach2 移出 src/ + ivg 标准分包重构 + peach 许可令牌余量语义调整 + 8090 日志面板
- peach2 十二包移出 src/（冻结归档 _archive/parked_2026-10-12/peach2/，本地留档）；AGENTS.md/CLAUDE.md/测试指导口径同轮收口为单入口
- ivg 对齐主流分包：tool_changer 的 URDF/meshes/tools.yaml 拆出 ivg_description，新增 ivg_bringup（ivg_system.launch.py）与 ivg_moveit_config（srdf/ompl/pilz）；ivg_sim 由 Allegro Hand 换 Original CAD 四爪夹爪（力命令非位置，单爪可被接触截停）+ gripper_contact 仿真夹具与冒烟；demo_services/latte_backend/graspnet/web_dashboard 接线迁到新包
- peach 许可令牌：radial/axial 余量改为记录给机械对刀具常数（负值不再拦套入/剪切）；TOOL 档仍查预备位残差与 tool.enabled；Clearance/GraspDecision 注释、peach_arm cycle/target_cache、包文档同轮
- scene_obstacles：部署默认 enabled: false（真机枝叶快照封死套入走廊，关闭态触发只发 REMOVE 清场）+ 体素 0.06→0.12；test_scene_obstacles 显式 enabled: true 并钉 0.06 体素（断言按半体素容差写死）
- 8090：新增 /api/state.logs 节点日志环形缓冲（log_buffer_size 参数、级别阈值+节点名过滤）与面板缓冲全量滚动；peach_web 补 web_state.test.cjs
- runs/ 过程文本层（账本/events/selfcheck，二进制仍本地）与 weights/yolo26n.pt（5.3MB）入库

验证：colcon build 35 包全过（含新增 ivg 三包）；受影响包 colcon test 绿（scene_obstacles 3/3）；interface manifest 57+5 核对通过。e1_supervisor_chain 为改动前已存在的 rviz2 无头环境红（09:36/09:59 复现于本轮改动前），非本轮引入。

File: src/ivg/ivg_sim/urdf/aubo_e5_ivg_sim.xacro (robot description, xacro)
@@ -1,26 +1,11 @@
 <?xml version="1.0"?>
-<!--
-  ivg_sim 抓取执行机器人 v3（2026-09-30）：原厂 AUBO E5 + 原装四指夹爪
-  （tool_changer 电动夹爪 φ60，gripper2 剖分）+ 仿真基座 + gz_ros2_control。
-  v1→v3 变更：v1 自制两指爪装配错位（用户指正）；v2 barista 整模换装在
-  gz 中观感碎块化（SW 多色分件 STL）+ 零位侧伸（用户指正）；v3 回原厂臂，
-  四指爪按 tool_changer 原装装配链挂接——
-    wrist3 →(0,0,0.020)→ camera_Link →(0,0,0.0215, Rz π)→ kuaihuan
-    →(0,0,0.020)→ gripper2
-  三段合成 = g2_base_joint：xyz (0,0,0.0615) rpy (0,0,π)。
-  四指 = gripper2 网格剖分（scripts/split_gripper2.py）：闭态十字排布，
-  径向 prismatic 同步开合（行程 55mm → 开口 119×138mm）。四向同步闭合
-  自定心，治两指先触指推飞问题。
-  TCP=指端包络腔心 = 法兰下 0.0615+0.175=0.2365 m；姿态恒等
-  （Z=approach、X=宽度，与 graspnet_to_ros_rotation 对齐）。
-  ros2_control 为本包自有声明（驱动栈只读）；world link/world_joint 由
-  arm_description.strip_world() 在 launch 侧剥除（gz 浮基 spawn）。
--->
 <robot name="aubo_e5" xmlns:xacro="http://www.ros.org/wiki/xacro">
-  <xacro:include filename="$(find aubo_description)/urdf/aubo_e5.urdf"/>
-  <!-- ======================= 仿真基座（重力世界锚定） ======================= -->
-  <!-- 宽 0.24：基座心 x=-0.58（SPAWN_XYZ 单源）时前缘 -0.46 距桌沿（-0.45）
-       1cm 不相交（MoveIt 永碰撞态红线），且抗前倾矩 353 Nm > 全展 223 Nm；
-       0.18 窄基座曾在全展抓取时整体前翻（2026-09-30 实测） -->
+<xacro:arg name="gripper" default="gripper2"/>
+<xacro:include filename="$(find ivg_description)/urdf/base.xacro"/>
+<xacro:include filename="$(find ivg_description)/urdf/tools.xacro"/>
+<xacro:include filename="$(find ivg_description)/urdf/gripper2_sim.xacro"/>
+<xacro:ivg_base include_workcell="false"/>
+<xacro:ivg_tools gripper="$(arg gripper)" tools_file="$(find ivg_description)/config/tools.yaml" articulated="true"/>
+<xacro:ivg_gripper2_fingers/>
   <link name="pedestal_link">
     <inertial>
@@ -44,24 +29,4 @@
     <origin xyz="0 0 -0.375" rpy="0 0 0"/>
   </joint>
-  <!-- ======================= Allegro Hand（社区常用四指手，仅仿真） =======================
-       源：felixduvallet/allegro-hand-ros allegro_hand_description（右手，
-       vendor 于 urdf/allegro_hand.xacro + meshes/allegro/）；16 revolute
-       关节（四指×4：外展/近/中/远节），自带 damping/friction（断电自锁）。
-       用户裁定（2026-09-30）：换社区常用四指夹爪（Robotiq 2F-140 两指
-       与 gripper2 剖分爪先后退场）。挂 wrist3，手指沿 +z（工具方向）。 -->
-  <xacro:include filename="$(find ivg_sim)/urdf/allegro_hand.xacro"/>
-  <joint name="allegro_mount_joint" type="fixed">
-    <parent link="wrist3_Link"/>
-    <child link="hand_root"/>
-    <origin xyz="0 0 0.02" rpy="0 0 0"/>
-  </joint>
-  <!-- ======================= 腕上相机（eye-in-hand，标定外参+内参） =======================
-       外参：aubo_hand_eye_calibration/hand_eye/active.yaml（已激活，
-       eye_in_hand，RMS 3.19mm）。光学帧 wrist3 直挂（scipy 核定 rpy）。
-       camera_mount 为 gz 传感器挂体（gz 点云轴系实测=body：x=视轴；
-       mount rpy 由外参合成，光轴沿工具方向）。
-       内参：percipio_camera/config/color_camera_info.yaml：fx=466.17
-       → hfov=1.203132；k1=0.0037 近零；center 0.5095/0.5100 未建模
-       （gz distortion 中心归一化近似 0.5，偏移 0.9% 影响可忽略）。 -->
   <link name="camera_mount_link">
     <inertial>
@@ -103,175 +68,16 @@
     </sensor>
   </gazebo>
-  <!-- TCP：Allegro 抓取腔心。掌面 hand_root+0.095，指全长 ~0.148
-       （tip ~0.243）；抓取腔心取 hand_root+0.203（≈指尖下 4cm，
-       对象上部包络区；spawn 后 TF 校核微调）。姿态与 wrist3 恒等。 -->
-  <link name="tcp">
-    <inertial>
-      <origin xyz="0 0 0" rpy="0 0 0"/>
-      <mass value="0.001"/>
-      <inertia ixx="1e-6" ixy="0" ixz="0" iyy="1e-6" iyz="0" izz="1e-6"/>
-    </inertial>
-  </link>
-  <joint name="tcp_joint" type="fixed">
-    <parent link="hand_root"/>
-    <child link="tcp"/>
-    <origin xyz="0 0 0.203" rpy="0 0 0"/>
-  </joint>
-  <!-- ======================= gz_ros2_control（本包自有声明） ======================= -->
-  <ros2_control name="IvgSimGazeboSystem" type="system">
-    <hardware>
-      <plugin>gz_ros2_control/GazeboSimSystem</plugin>
-    </hardware>
-    <joint name="shoulder_joint">
-      <command_interface name="position"/>
-      <state_interface name="position"/>
-      <state_interface name="velocity"/>
-    </joint>
-    <joint name="upperArm_joint">
-      <command_interface name="position"/>
-      <state_interface name="position"/>
-      <state_interface name="velocity"/>
-    </joint>
-    <joint name="foreArm_joint">
-      <command_interface name="position"/>
-      <state_interface name="position"/>
-      <state_interface name="velocity"/>
-    </joint>
-    <joint name="wrist1_joint">
-      <command_interface name="position"/>
-      <state_interface name="position"/>
-      <state_interface name="velocity"/>
-    </joint>
-    <joint name="wrist2_joint">
-      <command_interface name="position"/>
-      <state_interface name="position"/>
-      <state_interface name="velocity"/>
-    </joint>
-    <joint name="wrist3_joint">
-      <command_interface name="position"/>
-      <state_interface name="position"/>
-      <state_interface name="velocity"/>
-    </joint>
-    <!-- Allegro 16 关节（四指×4）：全部 position 命令位；initial_value
-         = 张开位（断电自锁由原包 damping/friction 保证） -->
-    <joint name="joint_0">
-      <command_interface name="position"/>
-      <state_interface name="position">
-        <param name="initial_value">0.0</param>
-      </state_interface>
-      <state_interface name="velocity"/>
-    </joint>
-    <joint name="joint_1">
-      <command_interface name="position"/>
-      <state_interface name="position">
-        <param name="initial_value">0.0</param>
-      </state_interface>
-      <state_interface name="velocity"/>
-    </joint>
-    <joint name="joint_2">
-      <command_interface name="position"/>
-      <state_interface name="position">
-        <param name="initial_value">0.0</param>
-      </state_interface>
-      <state_interface name="velocity"/>
-    </joint>
-    <joint name="joint_3">
-      <command_interface name="position"/>
-      <state_interface name="position">
-        <param name="initial_value">0.0</param>
-      </state_interface>
-      <state_interface name="velocity"/>
-    </joint>
-    <joint name="joint_4">
-      <command_interface name="position"/>
-      <state_interface name="position">
-        <param name="initial_value">0.0</param>
-      </state_interface>
-      <state_interface name="velocity"/>
-    </joint>
-    <joint name="joint_5">
-      <command_interface name="position"/>
-      <state_interface name="position">
-        <param name="initial_value">0.0</param>
-      </state_interface>
-      <state_interface name="velocity"/>
-    </joint>
-    <joint name="joint_6">
-      <command_interface name="position"/>
-      <state_interface name="position">
-        <param name="initial_value">0.0</param>
-      </state_interface>
-      <state_interface name="velocity"/>
-    </joint>
-    <joint name="joint_7">
-      <command_interface name="position"/>
-      <state_interface name="position">
-        <param name="initial_value">0.0</param>
-      </state_interface>
-      <state_interface name="velocity"/>
-    </joint>
-    <joint name="joint_8">
-      <command_interface name="position"/>
-      <state_interface name="position">
-        <param name="initial_value">0.0</param>
-      </state_interface>
-      <state_interface name="velocity"/>
-    </joint>
-    <joint name="joint_9">
-      <command_interface name="position"/>
-      <state_interface name="position">
-        <param name="initial_value">0.0</param>
-      </state_interface>
-      <state_interface name="velocity"/>
-    </joint>
-    <joint name="joint_10">
-      <command_interface name="position"/>
-      <state_interface name="position">
-        <param name="initial_value">0.0</param>
-      </state_interface>
-      <state_interface name="velocity"/>
-    </joint>
-    <joint name="joint_11">
-      <command_interface name="position"/>
-      <state_interface name="position">
-        <param name="initial_value">0.0</param>
-      </state_interface>
-      <state_interface name="velocity"/>
-    </joint>
-    <joint name="joint_12">
-      <command_interface name="position"/>
-      <state_interface name="position">
-        <param name="initial_value">0.3</param>
-      </state_interface>
-      <state_interface name="velocity"/>
-    </joint>
-    <joint name="joint_13">
-      <command_interface name="position"/>
-      <state_interface name="position">
-        <param name="initial_value">0.0</param>
-      </state_interface>
-      <state_interface name="velocity"/>
-    </joint>
-    <joint name="joint_14">
-      <command_interface name="position"/>
-      <state_interface name="position">
-        <param name="initial_value">0.0</param>
-      </state_interface>
-      <state_interface name="velocity"/>
-    </joint>
-    <joint name="joint_15">
-      <command_interface name="position"/>
-      <state_interface name="position">
-        <param name="initial_value">0.0</param>
-      </state_interface>
-      <state_interface name="velocity"/>
-    </joint>
-  </ros2_control>
-  <gazebo>
-    <plugin filename="gz_ros2_control-system" name="gz_ros2_control::GazeboSimROS2ControlPlugin">
-      <parameters>$(find ivg_sim)/config/gz_controllers.yaml</parameters>
-      <robot_param>robot_description</robot_param>
-      <robot_param_node>robot_state_publisher</robot_param_node>
-    </plugin>
-  </gazebo>
+<ros2_control name="IvgSimGazeboSystem" type="system"><hardware><plugin>gz_ros2_control/GazeboSimSystem</plugin></hardware>
+<joint name="shoulder_joint"><command_interface name="position"/><state_interface name="position"/><state_interface name="velocity"/></joint>
+<joint name="upperArm_joint"><command_interface name="position"/><state_interface name="position"/><state_interface name="velocity"/></joint>
+<joint name="foreArm_joint"><command_interface name="position"/><state_interface name="position"/><state_interface name="velocity"/></joint>
+<joint name="wrist1_joint"><command_interface name="position"/><state_interface name="position"/><state_interface name="velocity"/></joint>
+<joint name="wrist2_joint"><command_interface name="position"/><state_interface name="position"/><state_interface name="velocity"/></joint>
+<joint name="wrist3_joint"><command_interface name="position"/><state_interface name="position"/><state_interface name="velocity"/></joint>
+<joint name="gripper2_pp_joint"><command_interface name="effort"><param name="min">-20</param><param name="max">20</param></command_interface><state_interface name="position"><param name="initial_value">0.055</param></state_interface><state_interface name="velocity"/><state_interface name="effort"/></joint>
+<joint name="gripper2_pn_joint"><command_interface name="effort"><param name="min">-20</param><param name="max">20</param></command_interface><state_interface name="position"><param name="initial_value">0.055</param></state_interface><state_interface name="velocity"/><state_interface name="effort"/></joint>
+<joint name="gripper2_np_joint"><command_interface name="effort"><param name="min">-20</param><param name="max">20</param></command_interface><state_interface name="position"><param name="initial_value">0.055</param></state_interface><state_interface name="velocity"/><state_interface name="effort"/></joint>
+<joint name="gripper2_nn_joint"><command_interface name="effort"><param name="min">-20</param><param name="max">20</param></command_interface><state_interface name="position"><param name="initial_value">0.055</param></state_interface><state_interface name="velocity"/><state_interface name="effort"/></joint>
+</ros2_control>
+<gazebo><plugin filename="libgz_ros2_control-system.so" name="gz_ros2_control::GazeboSimROS2ControlPlugin"><parameters>$(find ivg_sim)/config/gz_controllers.yaml</parameters><hold_joints>true</hold_joints></plugin></gazebo>
 </robot>

File: src/ivg/tool_changer/urdf/aubo_e5_base.urdf (robot description, URDF)
Before this commit: robot aubo_e5, 15 links, 14 joints
Links:
- link camera_Link: geometry collision mesh filename=package://ivg_description/meshes/collision/camera_link.stl; visual mesh filename=package://ivg_description/meshes/visual/camera_link.stl
- link coffee_Link: geometry collision mesh filename=package://ivg_description/meshes/collision/coffee_link.stl; visual mesh filename=package://ivg_description/meshes/visual/coffee_link.stl
- link cup0_Link: geometry collision mesh filename=package://ivg_description/meshes/collision/cup0_link.stl; visual mesh filename=package://ivg_description/meshes/visual/cup0_link.stl
- link kuaihuan_Link: geometry collision mesh filename=package://ivg_description/meshes/collision/kuaihuan_link.stl; visual mesh filename=package://ivg_description/meshes/visual/kuaihuan_link.stl
- link lizhu_Link: geometry collision mesh filename=package://ivg_description/meshes/collision/lizhu_link.stl; visual mesh filename=package://ivg_description/meshes/visual/lizhu_link.stl
- link pedestal_Link: geometry collision mesh filename=package://ivg_description/meshes/collision/pedestal_link.stl; visual mesh filename=package://ivg_description/meshes/visual/pedestal_link.stl

File: src/ivg/tool_changer/urdf/aubo_e5_gripper0.urdf (robot description, URDF)
Before this commit: robot aubo_e5, 16 links, 15 joints
Links:
- link camera_Link: geometry collision mesh filename=package://ivg_description/meshes/collision/camera_link.stl; visual mesh filename=package://ivg_description/meshes/visual/camera_link.stl
- link coffee_Link: geometry collision mesh filename=package://ivg_description/meshes/collision/coffee_link.stl; visual mesh filename=package://ivg_description/meshes/visual/coffee_link.stl
- link cup0_Link: geometry collision mesh filename=package://ivg_description/meshes/collision/cup0_link.stl; visual mesh filename=package://ivg_description/meshes/visual/cup0_link.stl
- link gripper0_Link: geometry collision mesh filename=package://ivg_description/meshes/collision/gripper0_link.stl; visual mesh filename=package://ivg_description/meshes/visual/gripper0_link.stl
- link kuaihuan_Link: geometry collision mesh filename=package://ivg_description/meshes/collision/kuaihuan_link.stl; visual mesh filename=package://ivg_description/meshes/visual/kuaihuan_link.stl
- link lizhu_Link: geometry collision mesh filename=package://ivg_description/meshes/collision/lizhu_link.stl; visual mesh filename=package://ivg_description/meshes/visual/lizhu_link.stl
- link pedestal_Link: geometry collision mesh filename=package://ivg_description/meshes/collision/pedestal_link.stl; visual mesh filename=package://ivg_description/meshes/visual/pedestal_link.stl

File: src/ivg/tool_changer/urdf/aubo_e5_gripper1.urdf (robot description, URDF)
Before this commit: robot aubo_e5, 16 links, 15 joints
Links:
- link camera_Link: geometry collision mesh filename=package://ivg_description/meshes/collision/camera_link.stl; visual mesh filename=package://ivg_description/meshes/visual/camera_link.stl
- link coffee_Link: geometry collision mesh filename=package://ivg_description/meshes/collision/coffee_link.stl; visual mesh filename=package://ivg_description/meshes/visual/coffee_link.stl
- link cup0_Link: geometry collision mesh filename=package://ivg_description/meshes/collision/cup0_link.stl; visual mesh filename=package://ivg_description/meshes/visual/cup0_link.stl
- link gripper1_Link: geometry collision mesh filename=package://ivg_description/meshes/collision/gripper1_link.stl; visual mesh filename=package://ivg_description/meshes/visual/gripper1_link.stl
- link kuaihuan_Link: geometry collision mesh filename=package://ivg_description/meshes/collision/kuaihuan_link.stl; visual mesh filename=package://ivg_description/meshes/visual/kuaihuan_link.stl
- link lizhu_Link: geometry collision mesh filename=package://ivg_description/meshes/collision/lizhu_link.stl; visual mesh filename=package://ivg_description/meshes/visual/lizhu_link.stl
- link pedestal_Link: geometry collision mesh filename=package://ivg_description/meshes/collision/pedestal_link.stl; visual mesh filename=package://ivg_description/meshes/visual/pedestal_link.stl

File: src/ivg/tool_changer/urdf/aubo_e5_gripper1coffeecup.urdf (robot description, URDF)
Before this commit: robot aubo_e5, 16 links, 15 joints
Links:
- link camera_Link: geometry collision mesh filename=package://ivg_description/meshes/collision/camera_link.stl; visual mesh filename=package://ivg_description/meshes/visual/camera_link.stl
- link coffee_Link: geometry collision mesh filename=package://ivg_description/meshes/collision/coffee_link.stl; visual mesh filename=package://ivg_description/meshes/visual/coffee_link.stl
- link cup0_Link: geometry collision mesh filename=package://ivg_description/meshes/collision/cup0_link.stl; visual mesh filename=package://ivg_description/meshes/visual/cup0_link.stl
- link gripper1coffeecup_Link: geometry collision mesh filename=package://ivg_description/meshes/collision/gripper1coffeecu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; visual mesh filename=package://ivg_description/meshes/visual/gripper1coffeecup_l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
- link kuaihuan_Link: geometry collision mesh filename=package://ivg_description/meshes/collision/kuaihuan_link.stl; visual mesh filename=package://ivg_description/meshes/visual/kuaihuan_link.stl
- link lizhu_Link: geometry collision mesh filename=package://ivg_description/meshes/collision/lizhu_link.stl; visual mesh filename=package://ivg_description/meshes/visual/lizhu_link.stl
- link pedestal_Link: geometry collision mesh filename=package://ivg_description/meshes/collision/pedestal_link.stl; visual mesh filename=package://ivg_description/meshes/visual/pedestal_link.stl

File: src/ivg/tool_changer/urdf/aubo_e5_gripper1milkcup.urdf (robot description, URDF)
Before this commit: robot aubo_e5, 16 links, 15 joints
Links:
- link camera_Link: geometry collision mesh filename=package://ivg_description/meshes/collision/camera_link.stl; visual mesh filename=package://ivg_description/meshes/visual/camera_link.stl
- link coffee_Link: geometry collision mesh filename=package://ivg_description/meshes/collision/coffee_link.stl; visual mesh filename=package://ivg_description/meshes/visual/coffee_link.stl
- link cup0_Link: geometry collision mesh filename=package://ivg_description/meshes/collision/cup0_link.stl; visual mesh filename=package://ivg_description/meshes/visual/cup0_link.stl
- link gripper1milkcup_Link: geometry collision mesh filename=package://ivg_description/meshes/collision/gripper1milkcup_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; visual mesh filename=package://ivg_description/meshes/visual/gripper1milkcup_lin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
- link kuaihuan_Link: geometry collision mesh filename=package://ivg_description/meshes/collision/kuaihuan_link.stl; visual mesh filename=package://ivg_description/meshes/visual/kuaihuan_link.stl
- link lizhu_Link: geometry collision mesh filename=package://ivg_description/meshes/collision/lizhu_link.stl; visual mesh filename=package://ivg_description/meshes/visual/lizhu_link.stl
- link pedestal_Link: geometry collision mesh filename=package://ivg_description/meshes/collision/pedestal_link.stl; visual mesh filename=package://ivg_description/meshes/visual/pedestal_link.stl

File: src/ivg/tool_changer/urdf/aubo_e5_gripper2.urdf (robot description, URDF)
Before this commit: robot aubo_e5, 16 links, 15 joints
Links:
- link camera_Link: geometry collision mesh filename=package://ivg_description/meshes/collision/camera_link.stl; visual mesh filename=package://ivg_description/meshes/visual/camera_link.stl
- link coffee_Link: geometry collision mesh filename=package://ivg_description/meshes/collision/coffee_link.stl; visual mesh filename=package://ivg_description/meshes/visual/coffee_link.stl
- link cup0_Link: geometry collision mesh filename=package://ivg_description/meshes/collision/cup0_link.stl; visual mesh filename=package://ivg_description/meshes/visual/cup0_link.stl
- link gripper2_Link: geometry collision mesh filename=package://ivg_description/meshes/collision/gripper2_link.stl; visual mesh filename=package://ivg_description/meshes/visual/gripper2_link.stl
- link kuaihuan_Link: geometry collision mesh filename=package://ivg_description/meshes/collision/kuaihuan_link.stl; visual mesh filename=package://ivg_description/meshes/visual/kuaihuan_link.stl
- link lizhu_Link: geometry collision mesh filename=package://ivg_description/meshes/collision/lizhu_link.stl; visual mesh filename=package://ivg_description/meshes/visual/lizhu_link.stl
- link pedestal_Link: geometry collision mesh filename=package://ivg_description/meshes/collision/pedestal_link.stl; visual mesh filename=package://ivg_description/meshes/visual/pedestal_link.stl
