Commit message: feat(sim): P2 统一机体——gz_ros2_control 臂可控 + MoveIt + 可驾驶底盘一体
- sim_description/urdf/harvester_unified.urdf.xacro：单一模式根=platform_base_link，
  臂链拷贝自 aubo_e5.urdf（aubo_e5_arm.xacro 快照，掐掉 world_joint 世界锚定；
  mesh 仍 package://aubo_description 只读引用），base_link 经转台挂车体顶面 0.54m；
  相机帧链 = peach 感知契约（wrist3→camera_link 为手眼标定 active.yaml 快照，
  仿真单一 TF 源=RSP 不跑 extrinsics_publisher 叠帧）
- ros2_control：GazeboSimSystem 六关节 position 命令（config/gz_controllers.yaml
  JSB+JTC，use_sim_time）；/joint_states 由 JSB 原生发布（AUBO 六名/sim stamp）
- tracked_platform：chassis_visual 参数分离外观与可驾驶性（统一机体=BUNKER
  外观+DiffDrive 履带+桅杆激光）
- sim_bringup/sim.launch.py 主入口：作业位 spawn（0.95m，感知深度窗/臂展/
  photo_joints 标定位）；moveit:=true 复用 aubo_e5_moveit_config
  （controllers_file=controllers_mock.yaml，JTC 同名同关节零新映射）；
  spawner --service-call-timeout 60（重世界冷启动 CM 服务>10s，默认超时会撞
  already-loaded 卡 unconfigured，实测）
- field_no_grass.sdf 补不可见地面碰撞（统一机体在重建世界可落地）
- sim_system_tests：launch_testing 验收门（控制器双 active + /joint_states
  六 AUBO 名，isolated，300s 预算重世界首载）
- 已知：腕载 rgbd sensor 须挂 wrist3_Link 带 <pose>——空链 camera_link 的
  fixed-joint lump 会连 <gazebo> 扩展一起被 URDF→SDF 吞掉（scene/info 实证），
  xacro 注释在案
- 验收：结构测试 11/11；launch_testing 3/3；手动门全过（JTC 全关节目标
  shoulder→0.300rad 精确执行、cmd_vel 驾驶 odom 1.39m、move_group 四 action
  server 在册）

File: src/sim/sim_description/urdf/tracked_platform.xacro (robot description, xacro)
@@ -20,7 +20,11 @@
     数值入参一律字符串进、float() 出（xacro 属性默认是字符串，直接相加会拼接）。 -->
   <xacro:macro name="peach_tracked_platform"
-               params="parent arm_mount_height arm_mount_yaw_deg body_x body_y body_z body_bottom track_length track_width track_height track_separation mobile:=false">
+               params="parent arm_mount_height arm_mount_yaw_deg body_x body_y body_z body_bottom track_length track_width track_height track_separation mobile:=false chassis_visual:=''">
     <xacro:property name="mount_h" value="${float(arm_mount_height)}"/>
     <xacro:property name="mount_yaw" value="${-float(arm_mount_yaw_deg) * pi / 180.0}"/>
+    <!-- 车体外観：chassis_visual 显式覆盖（'bunker'|'box'）；空串跟随 mobile
+         （锚定=BUNKER 彩色网格，mobile=低模盒体）。统一机体 = bunker + 可驾驶。 -->
+    <xacro:property name="bunker_visual"
+                    value="${chassis_visual == 'bunker' or (chassis_visual == '' and not mobile)}"/>
     <xacro:property name="bx" value="${float(body_x)}"/>
     <xacro:property name="by" value="${float(body_y)}"/>
@@ -43,5 +47,5 @@
         <inertia ixx="4.05" ixy="0.0" ixz="0.0" iyy="12.05" iyz="0.0" izz="14.05"/>
       </inertial>
-      <xacro:unless value="${mobile}">
+      <xacro:if value="${bunker_visual}">
         <!-- BUNKER 外观网格：带颜色的车体/履带；碰撞仍用下面的简单代理。 -->
         <visual name="bunker_chassis_visual">
@@ -51,6 +55,6 @@
           </geometry>
         </visual>
-      </xacro:unless>
-      <xacro:if value="${mobile}">
+      </xacro:if>
+      <xacro:unless value="${bunker_visual}">
         <visual name="body_visual">
           <origin xyz="0 0 ${body_cz}" rpy="0 0 0"/>
@@ -62,5 +66,5 @@
           </material>
         </visual>
-      </xacro:if>
+      </xacro:unless>
       <collision name="body_collision">
         <origin xyz="0 0 ${body_cz}" rpy="0 0 0"/>
@@ -90,5 +94,6 @@
     </link>
     <!-- 层级：锚定 = world（臂座，模型根）→ platform_base_link → 履带/桅杆；
-       mobile = platform_base_link 即根（无臂链、无 world 链接） -->
+       mobile/统一机体 = platform_base_link 即根（无本关节；统一机体的臂由
+       外层挂到车体顶面） -->
     <xacro:unless value="${mobile}">
       <joint name="platform_mount" type="fixed">

Commit message: feat(sim): P4b 自主导航采摘——重建果园移植 + 底盘修正 + 感知域差桥接
== 重建果园移植（用户建模资产成为全链世界） ==
- field_gt.py 纯核：reconstruction scene_manifest → 树位/袋位/停靠位/导航地图
  （generate_field CLI；24 树/395 袋 GT，8 行×3 列，行距 3m 列距 5m）
- field_no_grass.sdf 补 Sensors(ogre2) 渲染系统 + 光照增亮（腕载 rgbd 可渲染）
- harvest.launch.py 一键全栈：sim(统一机体+MoveIt+相机) + perception + Nav2
  field 预设默认开启（field:=true；程序化世界 field:=false 保留为回归用）

== 底盘模型修正（对齐 AgileX 上游口径） ==
- VelocityControl 替代 DiffDrive：直接速度控制，不模拟轮子物理
  （上游 bunker_gazebo_sim 用 gazebo_ros_planar_move 同理）
- 履带碰撞：box 足迹 + 各向异性摩擦（替代圆柱滚筒 + 各向同性 μ=1）
  → 直线零侧滑（Δy=0.000m over 12.5m）零偏航（|Δyaw|<1e-9）
- odom_tf_relay.py：OdometryPublisher 的 gz 帧名（harvester/base_footprint）
  不可控，ROS 侧补 odom→platform_base_link TF 中继（标准 nav 模式）

== 感知域差桥接（gz-ogre2 vs Blender 渲染 → YOLO 分布） ==
- export_field_to_gz.py 烘纸袋 albedo 进 Base Color（修复前 gz 渲染无纸纹理
  → YOLO 零检出；烘后 conf 0.17-0.19 vs Blender 0.7+，检出解锁）
- sim_perception 阈值分叉：yolo_conf 0.35→0.12 / min_detection_conf 0.4→0.12 /
  confirm_frames 5→2 / min_collect_frames 10→60（gz 渲染域差 + worker 处理率
  0.5fps vs 到达 3.4Hz 的实测口径；真机 peach_harvester 保持原值）

== 自主采摘编排 ==
- orchard_harvest.py：逐站节拍 = stow 行驶→NavigateToPose→global_photo_pose→
  begin_scene→锁集→build_target_model→tcp 沿袋轴接近→stow
  SRDF 命名态自展开关节约束（MoveGroup action 不解析 Constraints.name）；
  epoch 过滤防旧窗竞态；有果站过滤（manifest reachable）；field stations-file
- sim.launch.py spawn_x/y/yaw 覆盖参数；goal_clearance 0.12m
- sim_harvest.rviz 13 层完整联合仿真视图

== Nav2 调优 ==
- inflation_radius 0.45→0.66（≥ 外接圆 0.642，官方口径）
- cost_scaling_factor 5.0→3.0（窄走廊平滑）
- AMCL alpha1-5 0.2→0.05（仿真里程计噪声收紧，防树行混叠跳变）
- MPPI vx_std 0.2→0.3 / wz_std 0.4→0.25 / vx_max 0.5→0.8

== 验收实跑（重建果园 3 站） ==
导航 3/3 到站（VelocityControl 底盘 100% 成功率）；
感知锁集 2 目标（target_0/target_1，累计命中 4760+ 持续增长）；
建模动作已发→重建采帧中（SAM 掩膜域差是最后一公里）

File: src/sim/sim_description/urdf/tracked_platform.xacro (robot description, xacro)
@@ -103,5 +103,5 @@
       </joint>
     </xacro:unless>
-    <xacro:macro name="track_unit" params="name side">
+      <xacro:macro name="track_unit" params="name side">
       <link name="${name}">
         <inertial>
@@ -121,11 +121,13 @@
           </visual>
         </xacro:if>
+        <!-- mobile（P4b 修正）：box 碰撞 = 履带接地印迹。VelocityControl
+             直接控制机体速度（对齐 AgileX planar_move 口径），不需要滚筒
+             物理滚动。圆柱滚筒方案实测侧滑 + MPPI 蛇形（各向同性 μ 下
+             横向无约束），2026-10-14 用户指出后修正。 -->
         <xacro:if value="${mobile}">
-          <!-- mobile：滚筒碰撞体（轴 Y、半径 th/2、长 tl）——DiffDrive 关节驱动下
-               平滑滚动，等效履带接地印迹；盒体仅作视觉 -->
           <collision name="${name}_collision">
-            <origin xyz="0 0 0" rpy="${pi / 2.0} 0 0"/>
+            <origin xyz="0 0 0" rpy="${pi / 2.0} 0 ${pi / 2.0}"/>
             <geometry>
-              <cylinder radius="${wheel_r}" length="${tl}"/>
+              <box size="${tw} ${th} ${tl}"/>
             </geometry>
           </collision>
@@ -139,74 +141,20 @@
           </collision>
         </xacro:unless>
-        <xacro:if value="${mobile}">
-          <visual name="${name}_wheel_front">
-            <origin xyz="${wheel_x} 0 0" rpy="${pi / 2.0} 0 0"/>
-            <geometry>
-              <cylinder radius="${wheel_r}" length="${tw}"/>
-            </geometry>
-            <material name="${name}_black"/>
-          </visual>
-        </xacro:if>
-        <collision name="${name}_wheel_front_collision">
-          <origin xyz="${wheel_x} 0 0" rpy="${pi / 2.0} 0 0"/>
-          <geometry>
-            <cylinder radius="${wheel_r}" length="${tw}"/>
-          </geometry>
-        </collision>
-        <xacro:if value="${mobile}">
-          <visual name="${name}_wheel_rear">
-            <origin xyz="${-wheel_x} 0 0" rpy="${pi / 2.0} 0 0"/>
-            <geometry>
-              <cylinder radius="${wheel_r}" length="${tw}"/>
-            </geometry>
-            <material name="${name}_black"/>
-          </visual>
-        </xacro:if>
-        <collision name="${name}_wheel_rear_collision">
-          <origin xyz="${-wheel_x} 0 0" rpy="${pi / 2.0} 0 0"/>
-          <geometry>
-            <cylinder radius="${wheel_r}" length="${tw}"/>
-          </geometry>
-        </collision>
       </link>
-      <!-- 履带挂接：mobile 用 continuous 转动关节当驱动轮——URDF→SDF 会把固定
-           关节子链接合并进父链接（fixed-joint lumping），履带不成其为独立链接、
-           无从驱动（冒烟实测固定关节时 TrackController 表面速度不出牵引）。
-           锚定模式仍用固定关节。 -->
-      <xacro:if value="${mobile}">
-        <joint name="${name}_mount" type="continuous">
-          <parent link="platform_base_link"/>
-          <child link="${name}"/>
-          <origin xyz="0 ${side * ts / 2.0} ${th / 2.0}" rpy="0 0 0"/>
-          <axis xyz="0 1 0"/>
-          <dynamics damping="0.05" friction="0.0"/>
-          <limit effort="1e5" velocity="20"/>
-        </joint>
-      </xacro:if>
-      <xacro:unless value="${mobile}">
-        <joint name="${name}_mount" type="fixed">
-          <parent link="platform_base_link"/>
-          <child link="${name}"/>
-          <origin xyz="0 ${side * ts / 2.0} ${th / 2.0}" rpy="0 0 0"/>
-        </joint>
-      </xacro:unless>
-      <!-- 履带摩擦：gz-physics dartsim 对未显式声明的碰撞不保证默认摩擦
-           （官方 TB3/TB4 轮子全部显式 <surface><friction>）。
-           mobile：各向同性 mu 1/1（TB3 轮口径，无 fdir1——圆柱碰撞系里
-           fdir1 会指向竖直方向、破坏滚动牵引，冒烟实测）。
-           锚定：官方履带口径（fdir1 车体横向 mu 0.7 / 纵向 mu2 150）。 -->
-      <xacro:if value="${mobile}">
-        <gazebo reference="${name}">
-          <mu1>1.0</mu1>
-          <mu2>1.0</mu2>
-        </gazebo>
-      </xacro:if>
-      <xacro:unless value="${mobile}">
-        <gazebo reference="${name}">
-          <mu1>0.7</mu1>
-          <mu2>150</mu2>
-          <fdir1>0 1 0</fdir1>
-        </gazebo>
-      </xacro:unless>
+      <!-- 履带挂接：统一用 fixed——VelocityControl 不需要旋转关节
+           （DiffDrive 需要 continuous 关节驱动滚筒；planar_move 口径下
+           履带只是碰撞足迹 + 视觉箱体）。 -->
+      <joint name="${name}_mount" type="fixed">
+        <parent link="platform_base_link"/>
+        <child link="${name}"/>
+        <origin xyz="0 ${side * ts / 2.0} ${th / 2.0}" rpy="0 0 0"/>
+      </joint>
+      <!-- 履带摩擦：统一用 box 各向异性——纵向低（前进阻力小）横向高
+           （抗侧滑，履带物理语义）。 -->
+      <gazebo reference="${name}">
+        <mu1>0.7</mu1>
+        <mu2>150</mu2>
+        <fdir1>0 1 0</fdir1>
+      </gazebo>
     </xacro:macro>
     <xacro:track_unit name="left_track" side="1.0"/>
@@ -283,26 +231,24 @@
         </sensor>
       </gazebo>
-      <!-- 底盘驱动：gz DiffDrive（官方 TB3/TB4 仿真同款，gz-sim 8 URDF 路径
-           验证可用）。左右履带 = 滚筒驱动轮（continuous 关节），odom 由关节
-           角积分。履带表面速度方案（TrackedVehicle+TrackController）在 8.15
-           URDF→SDF 路径上冒烟实测不出牵引（指令链通、整车不动），留待原生
-           SDF 模型轮再试。mobile 时转台偏航归零 → world 与 platform_base_link
-           同向，child_frame_id 取 platform_base_link 无恒定偏差。 -->
+      <!-- 底盘驱动（P4b 修正）：VelocityControl 直接控制机体速度（对齐 AgileX
+           planar_move 口径——上游 bunker_gazebo_sim 用 gazebo_ros_planar_move，
+           不模拟轮子物理，轮子仅视觉）。OdometryPublisher 从世界位姿发布
+           odom（无积分误差）。替换原 DiffDrive + 滚筒方案（各向同性 μ 下
+           侧滑 + MPPI 蛇形，2026-10-14 用户指出后修正）。 -->
       <gazebo>
-        <plugin name="gz::sim::systems::DiffDrive"
-                filename="gz-sim-diff-drive-system">
-          <left_joint>left_track_mount</left_joint>
-          <right_joint>right_track_mount</right_joint>
-          <wheel_separation>${ts}</wheel_separation>
-          <wheel_radius>${wheel_r}</wheel_radius>
+        <plugin name="gz::sim::systems::VelocityControl"
+                filename="gz-sim-velocity-control-system">
           <topic>/cmd_vel</topic>
+        </plugin>
+      </gazebo>
+      <gazebo>
+        <plugin name="gz::sim::systems::OdometryPublisher"
+                filename="gz-sim-odometry-publisher-system">
           <odom_topic>/odom</odom_topic>
+          <tf_topic>/tf</tf_topic>
+          <odom_frame>odom</odom_frame>
+          <robot_frame>platform_base_link</robot_frame>
           <odom_publish_frequency>50</odom_publish_frequency>
-          <tf_topic>/tf</tf_topic>
-          <frame_id>odom</frame_id>
-          <child_frame_id>platform_base_link</child_frame_id>
-          <max_linear_acceleration>1.0</max_linear_acceleration>
-          <max_linear_deceleration>1.0</max_linear_deceleration>
-          <max_angular_acceleration>2.0</max_angular_acceleration>
+          <dimensions>2</dimensions>
         </plugin>
       </gazebo>
